Commit message: action step 2, create base_link, laser_frame, imu_link

File: ros2_ws/src/robot_description/urdf/komatsu.urdf.xacro (robot description, xacro)
@@ -34,8 +34,17 @@
   <xacro:property name="box_w" value="${D_width-(2*wheel_width)}"/>
   <xacro:property name="box_h" value="${H_height-F_clearance}"/> <!-- just visual -->
+    <!-- base_footprint: ground projection of the robot -->
     <link name="base_footprint" />
+    <!-- base_link: main robot reference frame at articulation center -->
+    <link name="base_link"/>
+    <joint name="base_footprint_joint" type="fixed">
+        <parent link="base_footprint"/>
+        <child link="base_link"/>
+        <origin xyz="0 0 ${F_clearance}" rpy="0 0 0"/>
+    </joint>
+    <!-- articulation_link: center point of articulated steering -->
     <link name="articulation_link"/>
-    <joint name="base_joint" type="fixed">
-        <parent link="base_footprint"/>
+    <joint name="base_to_articulation_joint" type="fixed">
+        <parent link="base_link"/>
         <child link="articulation_link"/>
         <origin xyz="0 0 0" rpy="0 0 0"/>
@@ -81,3 +90,20 @@
   <xacro:wheel name="front_left_wheel"  parent="front_chassis" x="${ half_wb}" y="${ wheel_y}"/>
   <xacro:wheel name="front_right_wheel" parent="front_chassis" x="${ half_wb}" y="${-wheel_y}"/>
+  <!-- ===== Sensor Frames ===== -->
+  <!-- LiDAR sensor (mounted on top of front chassis, centered) -->
+  <link name="laser_frame"/>
+  <joint name="laser_joint" type="fixed">
+    <parent link="base_link"/>
+    <child link="laser_frame"/>
+    <!-- Position: on top of robot, centered -->
+    <origin xyz="0.0 0.0 ${H_height - F_clearance}" rpy="0 0 0"/>
+  </joint>
+  <!-- IMU sensor (mounted at base_link, centered) -->
+  <link name="imu_link"/>
+  <joint name="imu_joint" type="fixed">
+    <parent link="base_link"/>
+    <child link="imu_link"/>
+    <!-- Position: at base_link center -->
+    <origin xyz="0.0 0.0 0.0" rpy="0 0 0"/>
+  </joint>
 </robot>

Commit message: update turning angle

File: ros2_ws/src/robot_description/urdf/komatsu.urdf.xacro (robot description, xacro)
@@ -73,5 +73,5 @@
         <origin xyz="0 0 0" rpy="0 0 0"/>
         <axis xyz="0 0 1"/>
-        <limit lower="-0.392" upper="0.392" effort="5000" velocity="0.196"/>
+        <limit lower="-0.35" upper="0.35" effort="5000" velocity="0.196"/>
     </joint>
     <joint name="articulation_to_rear" type="revolute">
@@ -80,5 +80,5 @@
         <origin xyz="0 0 0" rpy="0 0 0"/>
         <axis xyz="0 0 1"/>
-        <limit lower="-0.392" upper="0.392" effort="5000" velocity="0.196"/>
+        <limit lower="-0.35" upper="0.35" effort="5000" velocity="0.196"/>
         <mimic joint="articulation_to_front" multiplier="-1" offset="0"/>
     </joint>

Commit message: gazebo integration

File: ros2_ws/src/robot_description/urdf/komatsu.urdf.xacro (robot description, xacro)
@@ -37,5 +37,11 @@
     <link name="base_footprint" />
     <!-- base_link: main robot reference frame at articulation center -->
-    <link name="base_link"/>
+    <link name="base_link">
+        <inertial>
+            <mass value="0.01"/>
+            <origin xyz="0 0 0" rpy="0 0 0"/>
+            <inertia ixx="0.001" ixy="0.0" ixz="0.0" iyy="0.001" iyz="0.0" izz="0.001"/>
+        </inertial>
+    </link>
     <joint name="base_footprint_joint" type="fixed">
         <parent link="base_footprint"/>
@@ -44,5 +50,11 @@
     </joint>
     <!-- articulation_link: center point of articulated steering -->
-    <link name="articulation_link"/>
+    <link name="articulation_link">
+        <inertial>
+            <mass value="0.01"/>
+            <origin xyz="0 0 0" rpy="0 0 0"/>
+            <inertia ixx="0.001" ixy="0.0" ixz="0.0" iyy="0.001" iyz="0.0" izz="0.001"/>
+        </inertial>
+    </link>
     <joint name="base_to_articulation_joint" type="fixed">
         <parent link="base_link"/>
@@ -58,4 +70,15 @@
             <material name="red"/>
         </visual>
+        <collision>
+            <origin xyz="${-rear_box_len/2.0} 0 ${F_clearance + box_h/2.0 - 0.10}" rpy="0 0 0"/>
+            <geometry>
+                <box size="${rear_box_len} ${box_w} ${box_h}"/>
+            </geometry>
+        </collision>
+        <inertial>
+            <mass value="5000.0"/>
+            <origin xyz="${-rear_box_len/2.0} 0 ${F_clearance + box_h/2.0 - 0.10}" rpy="0 0 0"/>
+            <inertia ixx="1000.0" ixy="0.0" ixz="0.0" iyy="2000.0" iyz="0.0" izz="1500.0"/>
+        </inertial>
     </link>
     <link name="front_chassis">
@@ -67,4 +90,15 @@
             <material name="green"/>
         </visual>
+        <collision>
+            <origin xyz="${front_box_len/2.0} 0 ${F_clearance + box_h/2.0 - 0.10}" rpy="0 0 0"/>
+            <geometry>
+                <box size="${front_box_len} ${box_w} ${box_h}"/>
+            </geometry>
+        </collision>
+        <inertial>
+            <mass value="5000.0"/>
+            <origin xyz="${front_box_len/2.0} 0 ${F_clearance + box_h/2.0 - 0.10}" rpy="0 0 0"/>
+            <inertia ixx="1000.0" ixy="0.0" ixz="0.0" iyy="2000.0" iyz="0.0" izz="1500.0"/>
+        </inertial>
     </link>
     <joint name="articulation_to_front" type="revolute">

File: ros2_ws/src/robot_description/urdf/wheels.xacro (robot description, xacro)
@@ -21,4 +21,15 @@
         <material name="black"/>
       </visual>
+      <collision>
+        <origin xyz="0 0 0" rpy="1.57079632679 0 0"/>
+        <geometry>
+          <cylinder radius="${radius}" length="${width}"/>
+        </geometry>
+      </collision>
+      <inertial>
+        <mass value="50.0"/>
+        <origin xyz="0 0 0" rpy="0 0 0"/>
+        <inertia ixx="5.0" ixy="0.0" ixz="0.0" iyy="10.0" iyz="0.0" izz="5.0"/>
+      </inertial>
     </link>
     <joint name="${name}_joint" type="continuous">

Commit message: create inertia as common property

File: ros2_ws/src/robot_description/urdf/komatsu.urdf.xacro (robot description, xacro)
@@ -1,6 +1,9 @@
 <?xml version="1.0"?>
 <robot name="komatsu" xmlns:xacro="http://www.ros.org/wiki/xacro">
+    <!-- Include common properties (inertia macros) -->
+    <xacro:include filename="$(find robot_description)/urdf/common_properties.xacro"/>
     <!-- Include wheel macro -->
     <xacro:include filename="$(find robot_description)/urdf/wheels.xacro"/>
+    <!-- Materials -->
     <material name="grey">
       <color rgba="0.7 0.7 0.7 1.0"/>
@@ -76,9 +79,10 @@
             </geometry>
         </collision>
-        <inertial>
-            <mass value="5000.0"/>
-            <origin xyz="${-rear_box_len/2.0} 0 ${F_clearance + box_h/2.0 - 0.10}" rpy="0 0 0"/>
-            <inertia ixx="1000.0" ixy="0.0" ixz="0.0" iyy="2000.0" iyz="0.0" izz="1500.0"/>
-        </inertial>
+        <xacro:box_inertia m="5000.0"
+                           x="${rear_box_len}"
+                           y="${box_w}"
+                           z="${box_h}"
+                           o_xyz="${-rear_box_len/2.0} 0 ${F_clearance + box_h/2.0 - 0.10}"
+                           o_rpy="0 0 0"/>
     </link>
     <link name="front_chassis">
@@ -96,9 +100,10 @@
             </geometry>
         </collision>
-        <inertial>
-            <mass value="5000.0"/>
-            <origin xyz="${front_box_len/2.0} 0 ${F_clearance + box_h/2.0 - 0.10}" rpy="0 0 0"/>
-            <inertia ixx="1000.0" ixy="0.0" ixz="0.0" iyy="2000.0" iyz="0.0" izz="1500.0"/>
-        </inertial>
+        <xacro:box_inertia m="5000.0"
+                           x="${front_box_len}"
+                           y="${box_w}"
+                           z="${box_h}"
+                           o_xyz="${front_box_len/2.0} 0 ${F_clearance + box_h/2.0 - 0.10}"
+                           o_rpy="0 0 0"/>
     </link>
     <joint name="articulation_to_front" type="revolute">

File: ros2_ws/src/robot_description/urdf/wheels.xacro (robot description, xacro)
@@ -11,4 +11,5 @@
       - radius: wheel radius (default: 0.80)
       - width: wheel width (default: 0.65)
+    Note: Requires cylinder_inertia macro from common_properties.xacro
   -->
   <xacro:macro name="wheel" params="name parent x y radius:=0.80 width:=0.65">
@@ -27,9 +28,9 @@
         </geometry>
       </collision>
-      <inertial>
-        <mass value="50.0"/>
-        <origin xyz="0 0 0" rpy="0 0 0"/>
-        <inertia ixx="5.0" ixy="0.0" ixz="0.0" iyy="10.0" iyz="0.0" izz="5.0"/>
-      </inertial>
+      <xacro:cylinder_inertia m="50.0"
+                              r="${radius}"
+                              l="${width}"
+                              o_xyz="0 0 0"
+                              o_rpy="0 0 0"/>
     </link>
     <joint name="${name}_joint" type="continuous">

Commit message: add base front and rear

File: ros2_ws/src/robot_description/urdf/komatsu.urdf.xacro (robot description, xacro)
@@ -1,43 +1,30 @@
 <?xml version="1.0"?>
 <robot name="komatsu" xmlns:xacro="http://www.ros.org/wiki/xacro">
-    <!-- Include common properties (inertia macros) -->
     <xacro:include filename="$(find robot_description)/urdf/common_properties.xacro"/>
-    <!-- Include wheel macro -->
     <xacro:include filename="$(find robot_description)/urdf/wheels.xacro"/>
-    <!-- Materials -->
-    <material name="grey">
-      <color rgba="0.7 0.7 0.7 1.0"/>
-    </material>
-    <material name="black">
-      <color rgba="0.1 0.1 0.1 1.0"/>
-    </material>
-    <material name="green">
-      <color rgba="0.0 1.0 0.0 1.0"/>
-    </material>
-    <material name="red">
-      <color rgba="1.0 0.0 0.0 1.0"/>
-    </material>
-  <!-- ===== Dimensions (meters) ===== -->
-  <xacro:property name="A_len" value="8.350"/>   <!-- Overall length -->
-  <xacro:property name="B_wheelbase" value="3.030"/> <!-- Wheelbase -->
-  <xacro:property name="D_width" value="2.765"/> <!-- Width over tires -->
-  <xacro:property name="E_track" value="2.160"/> <!-- Track width -->
-  <xacro:property name="F_clearance" value="0.455"/> <!-- Ground clearance -->
-  <xacro:property name="H_height" value="3.395"/> <!-- Overall height -->
-  <xacro:property name="X_len" value="3.200"/> <!-- Front overhang -->
-  <xacro:property name="Y_len" value="2.120"/> <!-- Rear overhang -->
-  <!-- Simplification choices -->
+    <material name="grey"><color rgba="0.7 0.7 0.7 1.0"/></material>
+    <material name="black"><color rgba="0.1 0.1 0.1 1.0"/></material>
+    <material name="green"><color rgba="0.0 1.0 0.0 1.0"/></material>
+    <material name="red"><color rgba="1.0 0.0 0.0 1.0"/></material>
+  <!-- ===== Dimensions ===== -->
+  <xacro:property name="A_len" value="8.350"/>
+  <xacro:property name="B_wheelbase" value="3.030"/>
+  <xacro:property name="D_width" value="2.765"/>
+  <xacro:property name="E_track" value="2.160"/>
+  <xacro:property name="F_clearance" value="0.455"/>
+  <xacro:property name="H_height" value="3.395"/>
+  <xacro:property name="X_len" value="3.200"/>
+  <xacro:property name="Y_len" value="2.120"/>
   <xacro:property name="half_wb" value="${B_wheelbase/2.0}"/>
-  <xacro:property name="wheel_radius" value="0.80"/>   <!-- approx (tire size 23.5 R25), adjust later -->
+  <xacro:property name="wheel_radius" value="0.80"/>
   <xacro:property name="wheel_width" value="0.65"/>
   <xacro:property name="wheel_y" value="${E_track/2.0}"/>
-  <!-- Two boxes (split overall length roughly in half) -->
   <xacro:property name="rear_box_len" value="${Y_len + half_wb}"/>
   <xacro:property name="front_box_len" value="${X_len + half_wb}"/>
   <xacro:property name="box_w" value="${D_width-(2*wheel_width)}"/>
-  <xacro:property name="box_h" value="${H_height-F_clearance}"/> <!-- just visual -->
-    <!-- base_footprint: ground projection of the robot -->
-    <link name="base_footprint" />
-    <!-- base_link: main robot reference frame at articulation center -->
+  <xacro:property name="box_h" value="${H_height-F_clearance}"/>
+    <!-- base footprint -->
+    <link name="base_footprint"/>
+    <!-- base link (articulation center reference) -->
     <link name="base_link">
         <inertial>
@@ -52,10 +39,10 @@
         <origin xyz="0 0 ${F_clearance}" rpy="0 0 0"/>
     </joint>
-    <!-- articulation_link: center point of articulated steering -->
+    <!-- articulation center -->
     <link name="articulation_link">
         <inertial>
             <mass value="0.01"/>
-            <origin xyz="0 0 0" rpy="0 0 0"/>
-            <inertia ixx="0.001" ixy="0.0" ixz="0.0" iyy="0.001" iyz="0.0" izz="0.001"/>
+            <origin xyz="0 0 0"/>
+            <inertia ixx="0.001" ixy="0" ixz="0" iyy="0.001" iyz="0" izz="0.001"/>
         </inertial>
     </link>
@@ -63,52 +50,47 @@
         <parent link="base_link"/>
         <child link="articulation_link"/>
-        <origin xyz="0 0 0" rpy="0 0 0"/>
     </joint>
+    <!-- rear body -->
     <link name="rear_chassis">
         <visual>
-            <origin xyz="${-rear_box_len/2.0} 0 ${F_clearance + box_h/2.0 - 0.10}" rpy="0 0 0"/>
-            <geometry>
-                <box size="${rear_box_len} ${box_w} ${box_h}"/>
-            </geometry>
+            <origin xyz="${-rear_box_len/2.0} 0 ${F_clearance + box_h/2.0 - 0.10}"/>
+            <geometry><box size="${rear_box_len} ${box_w} ${box_h}"/></geometry>
             <material name="red"/>
         </visual>
         <collision>
-            <origin xyz="${-rear_box_len/2.0} 0 ${F_clearance + box_h/2.0 - 0.10}" rpy="0 0 0"/>
-            <geometry>
-                <box size="${rear_box_len} ${box_w} ${box_h}"/>
-            </geometry>
+            <origin xyz="${-rear_box_len/2.0} 0 ${F_clearance + box_h/2.0 - 0.10}"/>
+            <geometry><box size="${rear_box_len} ${box_w} ${box_h}"/></geometry>
         </collision>
-        <xacro:box_inertia m="5000.0"
-                           x="${rear_box_len}"
-                           y="${box_w}"
-                           z="${box_h}"
-                           o_xyz="${-rear_box_len/2.0} 0 ${F_clearance + box_h/2.0 - 0.10}"
-                           o_rpy="0 0 0"/>
+        <xacro:box_inertia
+            m="5000.0"
+            x="${rear_box_len}"
+            y="${box_w}"
+            z="${box_h}"
+            o_xyz="${-rear_box_len/2.0} 0 ${F_clearance + box_h/2.0 - 0.10}"
+            o_rpy="0 0 0"/>
     </link>
+    <!-- front body -->
     <link name="front_chassis">
         <visual>
-            <origin xyz="${front_box_len/2.0} 0 ${F_clearance + box_h/2.0 - 0.10}" rpy="0 0 0"/>
-            <geometry>
-                <box size="${front_box_len} ${box_w} ${box_h}"/>
-            </geometry>
+            <origin xyz="${front_box_len/2.0} 0 ${F_clearance + box_h/2.0 - 0.10}"/>
+            <geometry><box size="${front_box_len} ${box_w} ${box_h}"/></geometry>
             <material name="green"/>
         </visual>
         <collision>
-            <origin xyz="${front_box_len/2.0} 0 ${F_clearance + box_h/2.0 - 0.10}" rpy="0 0 0"/>
-            <geometry>
-                <box size="${front_box_len} ${box_w} ${box_h}"/>
-            </geometry>
+            <origin xyz="${front_box_len/2.0} 0 ${F_clearance + box_h/2.0 - 0.10}"/>
+            <geometry><box size="${front_box_len} ${box_w} ${box_h}"/></geometry>
         </collision>
-        <xacro:box_inertia m="5000.0"
-                           x="${front_box_len}"
-                           y="${box_w}"
-                           z="${box_h}"
-                           o_xyz="${front_box_len/2.0} 0 ${F_clearance + box_h/2.0 - 0.10}"
-                           o_rpy="0 0 0"/>
+        <xacro:box_inertia
+            m="5000.0"
+            x="${front_box_len}"
+            y="${box_w}"
+            z="${box_h}"
+            o_xyz="${front_box_len/2.0} 0 ${F_clearance + box_h/2.0 - 0.10}"
+            o_rpy="0 0 0"/>
     </link>
+    <!-- articulation joints -->
     <joint name="articulation_to_front" type="revolute">
         <parent link="articulation_link"/>
         <child link="front_chassis"/>
-        <origin xyz="0 0 0" rpy="0 0 0"/>
         <axis xyz="0 0 1"/>
         <limit lower="-0.35" upper="0.35" effort="5000" velocity="0.196"/>
@@ -117,32 +99,38 @@
         <parent link="articulation_link"/>
         <child link="rear_chassis"/>
-        <origin xyz="0 0 0" rpy="0 0 0"/>
         <axis xyz="0 0 1"/>
         <limit lower="-0.35" upper="0.35" effort="5000" velocity="0.196"/>
-        <mimic joint="articulation_to_front" multiplier="-1" offset="0"/>
+        <mimic joint="articulation_to_front" multiplier="-1"/>
     </joint>
-  <!-- ===== Wheel macro is now in wheels.xacro ===== -->
-  <!-- ===== Rear axle wheels ===== -->
+  <!-- ===== Wheel macro ===== -->
   <xacro:wheel name="rear_left_wheel"  parent="rear_chassis" x="${-half_wb}" y="${ wheel_y}"/>
   <xacro:wheel name="rear_right_wheel" parent="rear_chassis" x="${-half_wb}" y="${-wheel_y}"/>
-  <!-- Front axle wheels (placed at x = +half_wb in front_chassis frame) -->
   <xacro:wheel name="front_left_wheel"  parent="front_chassis" x="${ half_wb}" y="${ wheel_y}"/>
   <xacro:wheel name="front_right_wheel" parent="front_chassis" x="${ half_wb}" y="${-wheel_y}"/>
-  <!-- ===== Sensor Frames ===== -->
-  <!-- LiDAR sensor (mounted on top of front chassis, centered) -->
+  <!-- ===== Navigation reference frames ===== -->
+  <link name="base_front"/>
+  <joint name="base_front_joint" type="fixed">
+    <parent link="front_chassis"/>
+    <child link="base_front"/>
+    <origin xyz="${half_wb} 0 0" rpy="0 0 0"/>
+  </joint>
+  <link name="base_rear"/>
+  <joint name="base_rear_joint" type="fixed">
+    <parent link="rear_chassis"/>
+    <child link="base_rear"/>
+    <origin xyz="${-half_wb} 0 0" rpy="0 0 0"/>
+  </joint>
+  <!-- ===== Sensors ===== -->
   <link name="laser_frame"/>
   <joint name="laser_joint" type="fixed">
-    <parent link="base_link"/>
+    <parent link="rear_chassis"/>
     <child link="laser_frame"/>
-    <!-- Position: on top of robot, centered -->
     <origin xyz="0.0 0.0 ${H_height - F_clearance}" rpy="0 0 0"/>
   </joint>
-  <!-- IMU sensor (mounted at base_link, centered) -->
   <link name="imu_link"/>
   <joint name="imu_joint" type="fixed">
     <parent link="base_link"/>
     <child link="imu_link"/>
-    <!-- Position: at base_link center -->
-    <origin xyz="0.0 0.0 0.0" rpy="0 0 0"/>
+    <origin xyz="0 0 0" rpy="0 0 0"/>
   </joint>
 </robot>

Commit message: adjust urdf

File: ros2_ws/src/robot_description/urdf/komatsu.urdf.xacro (robot description, xacro)
@@ -54,10 +54,10 @@
     <link name="rear_chassis">
         <visual>
-            <origin xyz="${-rear_box_len/2.0} 0 ${F_clearance + box_h/2.0 - 0.10}"/>
+            <origin xyz="${-rear_box_len/2.0} 0 ${box_h/2.0 - 0.10}"/>
             <geometry><box size="${rear_box_len} ${box_w} ${box_h}"/></geometry>
             <material name="red"/>
         </visual>
         <collision>
-            <origin xyz="${-rear_box_len/2.0} 0 ${F_clearance + box_h/2.0 - 0.10}"/>
+            <origin xyz="${-rear_box_len/2.0} 0 ${box_h/2.0 - 0.10}"/>
             <geometry><box size="${rear_box_len} ${box_w} ${box_h}"/></geometry>
         </collision>
@@ -67,5 +67,5 @@
             y="${box_w}"
             z="${box_h}"
-            o_xyz="${-rear_box_len/2.0} 0 ${F_clearance + box_h/2.0 - 0.10}"
+            o_xyz="${-rear_box_len/2.0} 0 ${box_h/2.0 - 0.10}"
             o_rpy="0 0 0"/>
     </link>
@@ -73,10 +73,10 @@
     <link name="front_chassis">
         <visual>
-            <origin xyz="${front_box_len/2.0} 0 ${F_clearance + box_h/2.0 - 0.10}"/>
+            <origin xyz="${front_box_len/2.0} 0 ${box_h/2.0 - 0.10}"/>
             <geometry><box size="${front_box_len} ${box_w} ${box_h}"/></geometry>
             <material name="green"/>
         </visual>
         <collision>
-            <origin xyz="${front_box_len/2.0} 0 ${F_clearance + box_h/2.0 - 0.10}"/>
+            <origin xyz="${front_box_len/2.0} 0 ${box_h/2.0 - 0.10}"/>
             <geometry><box size="${front_box_len} ${box_w} ${box_h}"/></geometry>
         </collision>
@@ -86,5 +86,5 @@
             y="${box_w}"
             z="${box_h}"
-            o_xyz="${front_box_len/2.0} 0 ${F_clearance + box_h/2.0 - 0.10}"
+            o_xyz="${front_box_len/2.0} 0 ${box_h/2.0 - 0.10}"
             o_rpy="0 0 0"/>
     </link>
@@ -126,5 +126,5 @@
     <parent link="rear_chassis"/>
     <child link="laser_frame"/>
-    <origin xyz="0.0 0.0 ${H_height - F_clearance}" rpy="0 0 0"/>
+    <origin xyz="0.0 0.0 ${box_h}" rpy="0 0 0"/>
   </joint>
   <link name="imu_link"/>

Commit message: adjust urdf

File: ros2_ws/src/robot_description/urdf/komatsu.urdf.xacro (robot description, xacro)
@@ -54,10 +54,10 @@
     <link name="rear_chassis">
         <visual>
-            <origin xyz="${-rear_box_len/2.0} 0 ${box_h/2.0 - 0.10}"/>
+            <origin xyz="${-rear_box_len/2.0} 0 ${box_h/2.0}"/>
             <geometry><box size="${rear_box_len} ${box_w} ${box_h}"/></geometry>
             <material name="red"/>
         </visual>
         <collision>
-            <origin xyz="${-rear_box_len/2.0} 0 ${box_h/2.0 - 0.10}"/>
+            <origin xyz="${-rear_box_len/2.0} 0 ${box_h/2.0}"/>
             <geometry><box size="${rear_box_len} ${box_w} ${box_h}"/></geometry>
         </collision>
@@ -67,5 +67,5 @@
             y="${box_w}"
             z="${box_h}"
-            o_xyz="${-rear_box_len/2.0} 0 ${box_h/2.0 - 0.10}"
+            o_xyz="${-rear_box_len/2.0} 0 ${box_h/2.0}"
             o_rpy="0 0 0"/>
     </link>
@@ -73,10 +73,10 @@
     <link name="front_chassis">
         <visual>
-            <origin xyz="${front_box_len/2.0} 0 ${box_h/2.0 - 0.10}"/>
+            <origin xyz="${front_box_len/2.0} 0 ${box_h/2.0}"/>
             <geometry><box size="${front_box_len} ${box_w} ${box_h}"/></geometry>
             <material name="green"/>
         </visual>
         <collision>
-            <origin xyz="${front_box_len/2.0} 0 ${box_h/2.0 - 0.10}"/>
+            <origin xyz="${front_box_len/2.0} 0 ${box_h/2.0}"/>
             <geometry><box size="${front_box_len} ${box_w} ${box_h}"/></geometry>
         </collision>
@@ -86,5 +86,5 @@
             y="${box_w}"
             z="${box_h}"
-            o_xyz="${front_box_len/2.0} 0 ${box_h/2.0 - 0.10}"
+            o_xyz="${front_box_len/2.0} 0 ${box_h/2.0}"
             o_rpy="0 0 0"/>
     </link>
