Commit message: adjust urdf 2

File: ros2_ws/src/robot_description/urdf/komatsu.urdf.xacro (robot description, xacro)
@@ -104,8 +104,8 @@
     </joint>
   <!-- ===== Wheel macro ===== -->
-  <xacro:wheel name="rear_left_wheel"  parent="rear_chassis" x="${-half_wb}" y="${ wheel_y}"/>
-  <xacro:wheel name="rear_right_wheel" parent="rear_chassis" x="${-half_wb}" y="${-wheel_y}"/>
-  <xacro:wheel name="front_left_wheel"  parent="front_chassis" x="${ half_wb}" y="${ wheel_y}"/>
-  <xacro:wheel name="front_right_wheel" parent="front_chassis" x="${ half_wb}" y="${-wheel_y}"/>
+  <xacro:wheel name="rear_left_wheel"  parent="rear_chassis" x="${-half_wb}" y="${ wheel_y}" z="${wheel_radius - F_clearance}"/>
+  <xacro:wheel name="rear_right_wheel" parent="rear_chassis" x="${-half_wb}" y="${-wheel_y}" z="${wheel_radius - F_clearance}"/>
+  <xacro:wheel name="front_left_wheel"  parent="front_chassis" x="${ half_wb}" y="${ wheel_y}" z="${wheel_radius - F_clearance}"/>
+  <xacro:wheel name="front_right_wheel" parent="front_chassis" x="${ half_wb}" y="${-wheel_y}" z="${wheel_radius - F_clearance}"/>
   <!-- ===== Navigation reference frames ===== -->
   <link name="base_front"/>
@@ -126,5 +126,5 @@
     <parent link="rear_chassis"/>
     <child link="laser_frame"/>
-    <origin xyz="0.0 0.0 ${box_h}" rpy="0 0 0"/>
+    <origin xyz="0.0 0.0 ${box_h + 0.03}" rpy="0 0 0"/>
   </joint>
   <link name="imu_link"/>

File: ros2_ws/src/robot_description/urdf/wheels.xacro (robot description, xacro)
@@ -9,9 +9,10 @@
       - x: x position relative to parent
       - y: y position relative to parent
+      - z: z position relative to parent (default: 0.80)
       - radius: wheel radius (default: 0.80)
       - width: wheel width (default: 0.65)
     Note: Requires cylinder_inertia macro from common_properties.xacro
   -->
-  <xacro:macro name="wheel" params="name parent x y radius:=0.80 width:=0.65">
+  <xacro:macro name="wheel" params="name parent x y z:=0.80 radius:=0.80 width:=0.65">
     <link name="${name}">
       <visual>
@@ -37,5 +38,5 @@
       <parent link="${parent}"/>
       <child link="${name}"/>
-      <origin xyz="${x} ${y} ${radius}" rpy="0 0 0"/>
+      <origin xyz="${x} ${y} ${z}" rpy="0 0 0"/>
       <!-- wheel rolls around Y (left axis), with ROS convention x forward, y left, z up -->
       <axis xyz="0 1 0"/>

Commit message: update urdf

File: ros2_ws/src/robot_description/urdf/komatsu.urdf.xacro (robot description, xacro)
@@ -37,5 +37,5 @@
         <parent link="base_footprint"/>
         <child link="base_link"/>
-        <origin xyz="0 0 ${F_clearance}" rpy="0 0 0"/>
+        <origin xyz="0 0 0" rpy="0 0 0"/>
     </joint>
     <!-- articulation center -->
@@ -54,10 +54,10 @@
     <link name="rear_chassis">
         <visual>
-            <origin xyz="${-rear_box_len/2.0} 0 ${box_h/2.0}"/>
+            <origin xyz="${-rear_box_len/2.0} 0 ${(box_h/2.0)+F_clearance}"/>
             <geometry><box size="${rear_box_len} ${box_w} ${box_h}"/></geometry>
             <material name="red"/>
         </visual>
         <collision>
-            <origin xyz="${-rear_box_len/2.0} 0 ${box_h/2.0}"/>
+            <origin xyz="${-rear_box_len/2.0} 0 ${(box_h/2.0)+F_clearance}"/>
             <geometry><box size="${rear_box_len} ${box_w} ${box_h}"/></geometry>
         </collision>
@@ -73,10 +73,10 @@
     <link name="front_chassis">
         <visual>
-            <origin xyz="${front_box_len/2.0} 0 ${box_h/2.0}"/>
+            <origin xyz="${front_box_len/2.0} 0 ${(box_h/2.0)+F_clearance}"/>
             <geometry><box size="${front_box_len} ${box_w} ${box_h}"/></geometry>
             <material name="green"/>
         </visual>
         <collision>
-            <origin xyz="${front_box_len/2.0} 0 ${box_h/2.0}"/>
+            <origin xyz="${front_box_len/2.0} 0 ${(box_h/2.0)+F_clearance}"/>
             <geometry><box size="${front_box_len} ${box_w} ${box_h}"/></geometry>
         </collision>
@@ -104,8 +104,8 @@
     </joint>
   <!-- ===== Wheel macro ===== -->
-  <xacro:wheel name="rear_left_wheel"  parent="rear_chassis" x="${-half_wb}" y="${ wheel_y}" z="${wheel_radius - F_clearance}"/>
-  <xacro:wheel name="rear_right_wheel" parent="rear_chassis" x="${-half_wb}" y="${-wheel_y}" z="${wheel_radius - F_clearance}"/>
-  <xacro:wheel name="front_left_wheel"  parent="front_chassis" x="${ half_wb}" y="${ wheel_y}" z="${wheel_radius - F_clearance}"/>
-  <xacro:wheel name="front_right_wheel" parent="front_chassis" x="${ half_wb}" y="${-wheel_y}" z="${wheel_radius - F_clearance}"/>
+  <xacro:wheel name="rear_left_wheel"  parent="rear_chassis" x="${-half_wb}" y="${ wheel_y}" z="${wheel_radius}"/>
+  <xacro:wheel name="rear_right_wheel" parent="rear_chassis" x="${-half_wb}" y="${-wheel_y}" z="${wheel_radius}"/>
+  <xacro:wheel name="front_left_wheel"  parent="front_chassis" x="${ half_wb}" y="${ wheel_y}" z="${wheel_radius}"/>
+  <xacro:wheel name="front_right_wheel" parent="front_chassis" x="${ half_wb}" y="${-wheel_y}" z="${wheel_radius}"/>
   <!-- ===== Navigation reference frames ===== -->
   <link name="base_front"/>

File: ros2_ws/src/robot_description/urdf/wheels.xacro (robot description, xacro)
@@ -14,5 +14,5 @@
     Note: Requires cylinder_inertia macro from common_properties.xacro
   -->
-  <xacro:macro name="wheel" params="name parent x y z:=0.80 radius:=0.80 width:=0.65">
+  <xacro:macro name="wheel" params="name parent x y z radius:=0.80 width:=0.65">
     <link name="${name}">
       <visual>

Commit message: Revert "update urdf"
This reverts commit 11f14e1bf848a48b184889d5173861e14124020b.

File: ros2_ws/src/robot_description/urdf/komatsu.urdf.xacro (robot description, xacro)
@@ -37,5 +37,5 @@
         <parent link="base_footprint"/>
         <child link="base_link"/>
-        <origin xyz="0 0 0" rpy="0 0 0"/>
+        <origin xyz="0 0 ${F_clearance}" rpy="0 0 0"/>
     </joint>
     <!-- articulation center -->
@@ -54,10 +54,10 @@
     <link name="rear_chassis">
         <visual>
-            <origin xyz="${-rear_box_len/2.0} 0 ${(box_h/2.0)+F_clearance}"/>
+            <origin xyz="${-rear_box_len/2.0} 0 ${box_h/2.0}"/>
             <geometry><box size="${rear_box_len} ${box_w} ${box_h}"/></geometry>
             <material name="red"/>
         </visual>
         <collision>
-            <origin xyz="${-rear_box_len/2.0} 0 ${(box_h/2.0)+F_clearance}"/>
+            <origin xyz="${-rear_box_len/2.0} 0 ${box_h/2.0}"/>
             <geometry><box size="${rear_box_len} ${box_w} ${box_h}"/></geometry>
         </collision>
@@ -73,10 +73,10 @@
     <link name="front_chassis">
         <visual>
-            <origin xyz="${front_box_len/2.0} 0 ${(box_h/2.0)+F_clearance}"/>
+            <origin xyz="${front_box_len/2.0} 0 ${box_h/2.0}"/>
             <geometry><box size="${front_box_len} ${box_w} ${box_h}"/></geometry>
             <material name="green"/>
         </visual>
         <collision>
-            <origin xyz="${front_box_len/2.0} 0 ${(box_h/2.0)+F_clearance}"/>
+            <origin xyz="${front_box_len/2.0} 0 ${box_h/2.0}"/>
             <geometry><box size="${front_box_len} ${box_w} ${box_h}"/></geometry>
         </collision>
@@ -104,8 +104,8 @@
     </joint>
   <!-- ===== Wheel macro ===== -->
-  <xacro:wheel name="rear_left_wheel"  parent="rear_chassis" x="${-half_wb}" y="${ wheel_y}" z="${wheel_radius}"/>
-  <xacro:wheel name="rear_right_wheel" parent="rear_chassis" x="${-half_wb}" y="${-wheel_y}" z="${wheel_radius}"/>
-  <xacro:wheel name="front_left_wheel"  parent="front_chassis" x="${ half_wb}" y="${ wheel_y}" z="${wheel_radius}"/>
-  <xacro:wheel name="front_right_wheel" parent="front_chassis" x="${ half_wb}" y="${-wheel_y}" z="${wheel_radius}"/>
+  <xacro:wheel name="rear_left_wheel"  parent="rear_chassis" x="${-half_wb}" y="${ wheel_y}" z="${wheel_radius - F_clearance}"/>
+  <xacro:wheel name="rear_right_wheel" parent="rear_chassis" x="${-half_wb}" y="${-wheel_y}" z="${wheel_radius - F_clearance}"/>
+  <xacro:wheel name="front_left_wheel"  parent="front_chassis" x="${ half_wb}" y="${ wheel_y}" z="${wheel_radius - F_clearance}"/>
+  <xacro:wheel name="front_right_wheel" parent="front_chassis" x="${ half_wb}" y="${-wheel_y}" z="${wheel_radius - F_clearance}"/>
   <!-- ===== Navigation reference frames ===== -->
   <link name="base_front"/>

File: ros2_ws/src/robot_description/urdf/wheels.xacro (robot description, xacro)
@@ -14,5 +14,5 @@
     Note: Requires cylinder_inertia macro from common_properties.xacro
   -->
-  <xacro:macro name="wheel" params="name parent x y z radius:=0.80 width:=0.65">
+  <xacro:macro name="wheel" params="name parent x y z:=0.80 radius:=0.80 width:=0.65">
     <link name="${name}">
       <visual>

Commit message: fix articulation

File: ros2_ws/src/robot_description/urdf/komatsu.urdf.xacro (robot description, xacro)
@@ -89,17 +89,17 @@
             o_rpy="0 0 0"/>
     </link>
-    <!-- articulation joints -->
+    <!-- rear chassis fixed to articulation center -->
+    <joint name="articulation_to_rear" type="fixed">
+        <parent link="articulation_link"/>
+        <child link="rear_chassis"/>
+        <origin xyz="0 0 0" rpy="0 0 0"/>
+    </joint>
+    <!-- single physical articulation joint -->
     <joint name="articulation_to_front" type="revolute">
         <parent link="articulation_link"/>
         <child link="front_chassis"/>
+        <origin xyz="0 0 0" rpy="0 0 0"/>
         <axis xyz="0 0 1"/>
         <limit lower="-0.35" upper="0.35" effort="5000" velocity="0.196"/>
-    </joint>
-    <joint name="articulation_to_rear" type="revolute">
-        <parent link="articulation_link"/>
-        <child link="rear_chassis"/>
-        <axis xyz="0 0 1"/>
-        <limit lower="-0.35" upper="0.35" effort="5000" velocity="0.196"/>
-        <mimic joint="articulation_to_front" multiplier="-1"/>
     </joint>
   <!-- ===== Wheel macro ===== -->

Commit message: add gnns, imu on rear body

File: ros2_ws/src/robot_description/urdf/komatsu.urdf.xacro (robot description, xacro)
@@ -122,15 +122,22 @@
   </joint>
   <!-- ===== Sensors ===== -->
+  <!-- Action_B: mount imu, gnss, laser on rear_chassis -->
   <link name="laser_frame"/>
   <joint name="laser_joint" type="fixed">
     <parent link="rear_chassis"/>
     <child link="laser_frame"/>
-    <origin xyz="0.0 0.0 ${box_h + 0.03}" rpy="0 0 0"/>
+    <origin xyz="0.0 0.0 ${box_h + 0.30}" rpy="0 0 0"/>
   </joint>
   <link name="imu_link"/>
   <joint name="imu_joint" type="fixed">
-    <parent link="base_link"/>
+    <parent link="rear_chassis"/>
     <child link="imu_link"/>
-    <origin xyz="0 0 0" rpy="0 0 0"/>
+    <origin xyz="0.0 0.0 ${box_h - 0.20}" rpy="0 0 0"/>
+  </joint>
+  <link name="gnss_link"/>
+  <joint name="gnss_joint" type="fixed">
+    <parent link="rear_chassis"/>
+    <child link="gnss_link"/>
+    <origin xyz="0.0 0.0 ${box_h - 0.10}" rpy="0 0 0"/>
   </joint>
 </robot>

Commit message: Revert "fix articulation"
This reverts commit 861d99dbe712bbc2abeecfacd572c5bf912d4fc8.

File: ros2_ws/src/robot_description/urdf/komatsu.urdf.xacro (robot description, xacro)
@@ -89,17 +89,17 @@
             o_rpy="0 0 0"/>
     </link>
-    <!-- rear chassis fixed to articulation center -->
-    <joint name="articulation_to_rear" type="fixed">
-        <parent link="articulation_link"/>
-        <child link="rear_chassis"/>
-        <origin xyz="0 0 0" rpy="0 0 0"/>
-    </joint>
-    <!-- single physical articulation joint -->
+    <!-- articulation joints -->
     <joint name="articulation_to_front" type="revolute">
         <parent link="articulation_link"/>
         <child link="front_chassis"/>
-        <origin xyz="0 0 0" rpy="0 0 0"/>
         <axis xyz="0 0 1"/>
         <limit lower="-0.35" upper="0.35" effort="5000" velocity="0.196"/>
+    </joint>
+    <joint name="articulation_to_rear" type="revolute">
+        <parent link="articulation_link"/>
+        <child link="rear_chassis"/>
+        <axis xyz="0 0 1"/>
+        <limit lower="-0.35" upper="0.35" effort="5000" velocity="0.196"/>
+        <mimic joint="articulation_to_front" multiplier="-1"/>
     </joint>
   <!-- ===== Wheel macro ===== -->

Commit message: disable articulation

File: ros2_ws/src/robot_description/urdf/komatsu.urdf.xacro (robot description, xacro)
@@ -7,24 +7,24 @@
     <material name="green"><color rgba="0.0 1.0 0.0 1.0"/></material>
     <material name="red"><color rgba="1.0 0.0 0.0 1.0"/></material>
-  <!-- ===== Dimensions ===== -->
-  <xacro:property name="A_len" value="8.350"/>
-  <xacro:property name="B_wheelbase" value="3.030"/>
-  <xacro:property name="D_width" value="2.765"/>
-  <xacro:property name="E_track" value="2.160"/>
-  <xacro:property name="F_clearance" value="0.455"/>
-  <xacro:property name="H_height" value="3.395"/>
-  <xacro:property name="X_len" value="3.200"/>
-  <xacro:property name="Y_len" value="2.120"/>
-  <xacro:property name="half_wb" value="${B_wheelbase/2.0}"/>
-  <xacro:property name="wheel_radius" value="0.80"/>
-  <xacro:property name="wheel_width" value="0.65"/>
-  <xacro:property name="wheel_y" value="${E_track/2.0}"/>
-  <xacro:property name="rear_box_len" value="${Y_len + half_wb}"/>
-  <xacro:property name="front_box_len" value="${X_len + half_wb}"/>
-  <xacro:property name="box_w" value="${D_width-(2*wheel_width)}"/>
-  <xacro:property name="box_h" value="${H_height-F_clearance}"/>
+    <!-- ===== Dimensions ===== -->
+    <xacro:property name="A_len" value="8.350"/>
+    <xacro:property name="B_wheelbase" value="3.030"/>
+    <xacro:property name="D_width" value="2.765"/>
+    <xacro:property name="E_track" value="2.160"/>
+    <xacro:property name="F_clearance" value="0.455"/>
+    <xacro:property name="H_height" value="3.395"/>
+    <xacro:property name="X_len" value="3.200"/>
+    <xacro:property name="Y_len" value="2.120"/>
+    <xacro:property name="half_wb" value="${B_wheelbase/2.0}"/>
+    <xacro:property name="wheel_radius" value="0.80"/>
+    <xacro:property name="wheel_width" value="0.65"/>
+    <xacro:property name="wheel_y" value="${E_track/2.0}"/>
+    <xacro:property name="rear_box_len" value="${Y_len + half_wb}"/>
+    <xacro:property name="front_box_len" value="${X_len + half_wb}"/>
+    <xacro:property name="box_w" value="${D_width-(2*wheel_width)}"/>
+    <xacro:property name="box_h" value="${H_height-F_clearance}"/>
     <!-- base footprint -->
     <link name="base_footprint"/>
-    <!-- base link (articulation center reference) -->
+    <!-- base link (vehicle reference) -->
     <link name="base_link">
         <inertial>
@@ -38,16 +38,4 @@
         <child link="base_link"/>
         <origin xyz="0 0 ${F_clearance}" rpy="0 0 0"/>
-    </joint>
-    <!-- articulation center -->
-    <link name="articulation_link">
-        <inertial>
-            <mass value="0.01"/>
-            <origin xyz="0 0 0"/>
-            <inertia ixx="0.001" ixy="0" ixz="0" iyy="0.001" iyz="0" izz="0.001"/>
-        </inertial>
-    </link>
-    <joint name="base_to_articulation_joint" type="fixed">
-        <parent link="base_link"/>
-        <child link="articulation_link"/>
     </joint>
     <!-- rear body -->
@@ -63,10 +51,10 @@
         </collision>
         <xacro:box_inertia
-            m="5000.0"
-            x="${rear_box_len}"
-            y="${box_w}"
-            z="${box_h}"
-            o_xyz="${-rear_box_len/2.0} 0 ${box_h/2.0}"
-            o_rpy="0 0 0"/>
+                m="5000.0"
+                x="${rear_box_len}"
+                y="${box_w}"
+                z="${box_h}"
+                o_xyz="${-rear_box_len/2.0} 0 ${box_h/2.0}"
+                o_rpy="0 0 0"/>
     </link>
     <!-- front body -->
@@ -82,55 +70,52 @@
         </collision>
         <xacro:box_inertia
-            m="5000.0"
-            x="${front_box_len}"
-            y="${box_w}"
-            z="${box_h}"
-            o_xyz="${front_box_len/2.0} 0 ${box_h/2.0}"
-            o_rpy="0 0 0"/>
+                m="5000.0"
+                x="${front_box_len}"
+                y="${box_w}"
+                z="${box_h}"
+                o_xyz="${front_box_len/2.0} 0 ${box_h/2.0}"
+                o_rpy="0 0 0"/>
     </link>
-    <!-- articulation joints -->
-    <joint name="articulation_to_front" type="revolute">
-        <parent link="articulation_link"/>
+    <!-- fixed chassis joints for quick Nav2 test -->
+    <joint name="base_to_front_joint" type="fixed">
+        <parent link="base_link"/>
         <child link="front_chassis"/>
-        <axis xyz="0 0 1"/>
-        <limit lower="-0.35" upper="0.35" effort="5000" velocity="0.196"/>
+        <origin xyz="0 0 0" rpy="0 0 0"/>
     </joint>
-    <joint name="articulation_to_rear" type="revolute">
-        <parent link="articulation_link"/>
+    <joint name="base_to_rear_joint" type="fixed">
+        <parent link="base_link"/>
         <child link="rear_chassis"/>
-        <axis xyz="0 0 1"/>
-        <limit lower="-0.35" upper="0.35" effort="5000" velocity="0.196"/>
-        <mimic joint="articulation_to_front" multiplier="-1"/>
+        <origin xyz="0 0 0" rpy="0 0 0"/>
     </joint>
-  <!-- ===== Wheel macro ===== -->
-  <xacro:wheel name="rear_left_wheel"  parent="rear_chassis" x="${-half_wb}" y="${ wheel_y}" z="${wheel_radius - F_clearance}"/>
-  <xacro:wheel name="rear_right_wheel" parent="rear_chassis" x="${-half_wb}" y="${-wheel_y}" z="${wheel_radius - F_clearance}"/>
-  <xacro:wheel name="front_left_wheel"  parent="front_chassis" x="${ half_wb}" y="${ wheel_y}" z="${wheel_radius - F_clearance}"/>
-  <xacro:wheel name="front_right_wheel" parent="front_chassis" x="${ half_wb}" y="${-wheel_y}" z="${wheel_radius - F_clearance}"/>
-  <!-- ===== Navigation reference frames ===== -->
-  <link name="base_front"/>
-  <joint name="base_front_joint" type="fixed">
-    <parent link="front_chassis"/>
-    <child link="base_front"/>
-    <origin xyz="${half_wb} 0 0" rpy="0 0 0"/>
-  </joint>
-  <link name="base_rear"/>
-  <joint name="base_rear_joint" type="fixed">
-    <parent link="rear_chassis"/>
-    <child link="base_rear"/>
-    <origin xyz="${-half_wb} 0 0" rpy="0 0 0"/>
-  </joint>
-  <!-- ===== Sensors ===== -->
-  <link name="laser_frame"/>
-  <joint name="laser_joint" type="fixed">
-    <parent link="rear_chassis"/>
-    <child link="laser_frame"/>
-    <origin xyz="0.0 0.0 ${box_h + 0.03}" rpy="0 0 0"/>
-  </joint>
-  <link name="imu_link"/>
-  <joint name="imu_joint" type="fixed">
-    <parent link="base_link"/>
-    <child link="imu_link"/>
-    <origin xyz="0 0 0" rpy="0 0 0"/>
-  </joint>
+    <!-- ===== Wheel macro ===== -->
+    <xacro:wheel name="rear_left_wheel"  parent="rear_chassis" x="${-half_wb}" y="${ wheel_y}" z="${wheel_radius - F_clearance}"/>
+    <xacro:wheel name="rear_right_wheel" parent="rear_chassis" x="${-half_wb}" y="${-wheel_y}" z="${wheel_radius - F_clearance}"/>
+    <xacro:wheel name="front_left_wheel"  parent="front_chassis" x="${ half_wb}" y="${ wheel_y}" z="${wheel_radius - F_clearance}"/>
+    <xacro:wheel name="front_right_wheel" parent="front_chassis" x="${ half_wb}" y="${-wheel_y}" z="${wheel_radius - F_clearance}"/>
+    <!-- ===== Navigation reference frames ===== -->
+    <link name="base_front"/>
+    <joint name="base_front_joint" type="fixed">
+        <parent link="front_chassis"/>
+        <child link="base_front"/>
+        <origin xyz="${half_wb} 0 0" rpy="0 0 0"/>
+    </joint>
+    <link name="base_rear"/>
+    <joint name="base_rear_joint" type="fixed">
+        <parent link="rear_chassis"/>
+        <child link="base_rear"/>
+        <origin xyz="${-half_wb} 0 0" rpy="0 0 0"/>
+    </joint>
+    <!-- ===== Sensors ===== -->
+    <link name="laser_frame"/>
+    <joint name="laser_joint" type="fixed">
+        <parent link="rear_chassis"/>
+        <child link="laser_frame"/>
+        <origin xyz="0.0 0.0 ${box_h + 0.03}" rpy="0 0 0"/>
+    </joint>
+    <link name="imu_link"/>
+    <joint name="imu_joint" type="fixed">
+        <parent link="base_link"/>
+        <child link="imu_link"/>
+        <origin xyz="0 0 0" rpy="0 0 0"/>
+    </joint>
 </robot>
