Commit message: Revert "disable articulation"
This reverts commit 0f5ffcbb179bcac26034b09835f634627adc1322.

File: ros2_ws/src/robot_description/urdf/komatsu.urdf.xacro (robot description, xacro)
@@ -7,24 +7,24 @@
     <material name="green"><color rgba="0.0 1.0 0.0 1.0"/></material>
     <material name="red"><color rgba="1.0 0.0 0.0 1.0"/></material>
-    <!-- ===== Dimensions ===== -->
-    <xacro:property name="A_len" value="8.350"/>
-    <xacro:property name="B_wheelbase" value="3.030"/>
-    <xacro:property name="D_width" value="2.765"/>
-    <xacro:property name="E_track" value="2.160"/>
-    <xacro:property name="F_clearance" value="0.455"/>
-    <xacro:property name="H_height" value="3.395"/>
-    <xacro:property name="X_len" value="3.200"/>
-    <xacro:property name="Y_len" value="2.120"/>
-    <xacro:property name="half_wb" value="${B_wheelbase/2.0}"/>
-    <xacro:property name="wheel_radius" value="0.80"/>
-    <xacro:property name="wheel_width" value="0.65"/>
-    <xacro:property name="wheel_y" value="${E_track/2.0}"/>
-    <xacro:property name="rear_box_len" value="${Y_len + half_wb}"/>
-    <xacro:property name="front_box_len" value="${X_len + half_wb}"/>
-    <xacro:property name="box_w" value="${D_width-(2*wheel_width)}"/>
-    <xacro:property name="box_h" value="${H_height-F_clearance}"/>
+  <!-- ===== Dimensions ===== -->
+  <xacro:property name="A_len" value="8.350"/>
+  <xacro:property name="B_wheelbase" value="3.030"/>
+  <xacro:property name="D_width" value="2.765"/>
+  <xacro:property name="E_track" value="2.160"/>
+  <xacro:property name="F_clearance" value="0.455"/>
+  <xacro:property name="H_height" value="3.395"/>
+  <xacro:property name="X_len" value="3.200"/>
+  <xacro:property name="Y_len" value="2.120"/>
+  <xacro:property name="half_wb" value="${B_wheelbase/2.0}"/>
+  <xacro:property name="wheel_radius" value="0.80"/>
+  <xacro:property name="wheel_width" value="0.65"/>
+  <xacro:property name="wheel_y" value="${E_track/2.0}"/>
+  <xacro:property name="rear_box_len" value="${Y_len + half_wb}"/>
+  <xacro:property name="front_box_len" value="${X_len + half_wb}"/>
+  <xacro:property name="box_w" value="${D_width-(2*wheel_width)}"/>
+  <xacro:property name="box_h" value="${H_height-F_clearance}"/>
     <!-- base footprint -->
     <link name="base_footprint"/>
-    <!-- base link (vehicle reference) -->
+    <!-- base link (articulation center reference) -->
     <link name="base_link">
         <inertial>
@@ -38,4 +38,16 @@
         <child link="base_link"/>
         <origin xyz="0 0 ${F_clearance}" rpy="0 0 0"/>
+    </joint>
+    <!-- articulation center -->
+    <link name="articulation_link">
+        <inertial>
+            <mass value="0.01"/>
+            <origin xyz="0 0 0"/>
+            <inertia ixx="0.001" ixy="0" ixz="0" iyy="0.001" iyz="0" izz="0.001"/>
+        </inertial>
+    </link>
+    <joint name="base_to_articulation_joint" type="fixed">
+        <parent link="base_link"/>
+        <child link="articulation_link"/>
     </joint>
     <!-- rear body -->
@@ -51,10 +63,10 @@
         </collision>
         <xacro:box_inertia
-                m="5000.0"
-                x="${rear_box_len}"
-                y="${box_w}"
-                z="${box_h}"
-                o_xyz="${-rear_box_len/2.0} 0 ${box_h/2.0}"
-                o_rpy="0 0 0"/>
+            m="5000.0"
+            x="${rear_box_len}"
+            y="${box_w}"
+            z="${box_h}"
+            o_xyz="${-rear_box_len/2.0} 0 ${box_h/2.0}"
+            o_rpy="0 0 0"/>
     </link>
     <!-- front body -->
@@ -70,52 +82,55 @@
         </collision>
         <xacro:box_inertia
-                m="5000.0"
-                x="${front_box_len}"
-                y="${box_w}"
-                z="${box_h}"
-                o_xyz="${front_box_len/2.0} 0 ${box_h/2.0}"
-                o_rpy="0 0 0"/>
+            m="5000.0"
+            x="${front_box_len}"
+            y="${box_w}"
+            z="${box_h}"
+            o_xyz="${front_box_len/2.0} 0 ${box_h/2.0}"
+            o_rpy="0 0 0"/>
     </link>
-    <!-- fixed chassis joints for quick Nav2 test -->
-    <joint name="base_to_front_joint" type="fixed">
-        <parent link="base_link"/>
+    <!-- articulation joints -->
+    <joint name="articulation_to_front" type="revolute">
+        <parent link="articulation_link"/>
         <child link="front_chassis"/>
-        <origin xyz="0 0 0" rpy="0 0 0"/>
+        <axis xyz="0 0 1"/>
+        <limit lower="-0.35" upper="0.35" effort="5000" velocity="0.196"/>
     </joint>
-    <joint name="base_to_rear_joint" type="fixed">
-        <parent link="base_link"/>
+    <joint name="articulation_to_rear" type="revolute">
+        <parent link="articulation_link"/>
         <child link="rear_chassis"/>
-        <origin xyz="0 0 0" rpy="0 0 0"/>
+        <axis xyz="0 0 1"/>
+        <limit lower="-0.35" upper="0.35" effort="5000" velocity="0.196"/>
+        <mimic joint="articulation_to_front" multiplier="-1"/>
     </joint>
-    <!-- ===== Wheel macro ===== -->
-    <xacro:wheel name="rear_left_wheel"  parent="rear_chassis" x="${-half_wb}" y="${ wheel_y}" z="${wheel_radius - F_clearance}"/>
-    <xacro:wheel name="rear_right_wheel" parent="rear_chassis" x="${-half_wb}" y="${-wheel_y}" z="${wheel_radius - F_clearance}"/>
-    <xacro:wheel name="front_left_wheel"  parent="front_chassis" x="${ half_wb}" y="${ wheel_y}" z="${wheel_radius - F_clearance}"/>
-    <xacro:wheel name="front_right_wheel" parent="front_chassis" x="${ half_wb}" y="${-wheel_y}" z="${wheel_radius - F_clearance}"/>
-    <!-- ===== Navigation reference frames ===== -->
-    <link name="base_front"/>
-    <joint name="base_front_joint" type="fixed">
-        <parent link="front_chassis"/>
-        <child link="base_front"/>
-        <origin xyz="${half_wb} 0 0" rpy="0 0 0"/>
-    </joint>
-    <link name="base_rear"/>
-    <joint name="base_rear_joint" type="fixed">
-        <parent link="rear_chassis"/>
-        <child link="base_rear"/>
-        <origin xyz="${-half_wb} 0 0" rpy="0 0 0"/>
-    </joint>
-    <!-- ===== Sensors ===== -->
-    <link name="laser_frame"/>
-    <joint name="laser_joint" type="fixed">
-        <parent link="rear_chassis"/>
-        <child link="laser_frame"/>
-        <origin xyz="0.0 0.0 ${box_h + 0.03}" rpy="0 0 0"/>
-    </joint>
-    <link name="imu_link"/>
-    <joint name="imu_joint" type="fixed">
-        <parent link="base_link"/>
-        <child link="imu_link"/>
-        <origin xyz="0 0 0" rpy="0 0 0"/>
-    </joint>
+  <!-- ===== Wheel macro ===== -->
+  <xacro:wheel name="rear_left_wheel"  parent="rear_chassis" x="${-half_wb}" y="${ wheel_y}" z="${wheel_radius - F_clearance}"/>
+  <xacro:wheel name="rear_right_wheel" parent="rear_chassis" x="${-half_wb}" y="${-wheel_y}" z="${wheel_radius - F_clearance}"/>
+  <xacro:wheel name="front_left_wheel"  parent="front_chassis" x="${ half_wb}" y="${ wheel_y}" z="${wheel_radius - F_clearance}"/>
+  <xacro:wheel name="front_right_wheel" parent="front_chassis" x="${ half_wb}" y="${-wheel_y}" z="${wheel_radius - F_clearance}"/>
+  <!-- ===== Navigation reference frames ===== -->
+  <link name="base_front"/>
+  <joint name="base_front_joint" type="fixed">
+    <parent link="front_chassis"/>
+    <child link="base_front"/>
+    <origin xyz="${half_wb} 0 0" rpy="0 0 0"/>
+  </joint>
+  <link name="base_rear"/>
+  <joint name="base_rear_joint" type="fixed">
+    <parent link="rear_chassis"/>
+    <child link="base_rear"/>
+    <origin xyz="${-half_wb} 0 0" rpy="0 0 0"/>
+  </joint>
+  <!-- ===== Sensors ===== -->
+  <link name="laser_frame"/>
+  <joint name="laser_joint" type="fixed">
+    <parent link="rear_chassis"/>
+    <child link="laser_frame"/>
+    <origin xyz="0.0 0.0 ${box_h + 0.03}" rpy="0 0 0"/>
+  </joint>
+  <link name="imu_link"/>
+  <joint name="imu_joint" type="fixed">
+    <parent link="base_link"/>
+    <child link="imu_link"/>
+    <origin xyz="0 0 0" rpy="0 0 0"/>
+  </joint>
 </robot>

Commit message: update urdf

File: ros2_ws/src/robot_description/urdf/komatsu.urdf.xacro (robot description, xacro)
@@ -14,6 +14,8 @@
   <xacro:property name="F_clearance" value="0.455"/>
   <xacro:property name="H_height" value="3.395"/>
-  <xacro:property name="X_len" value="3.200"/>
-  <xacro:property name="Y_len" value="2.120"/>
+  <xacro:property name="X_len" value="2.660"/>
+  <xacro:property name="Y_len" value="2.660"/>
+    <xacro:property name="HR_height" value="2.350"/> <!-- rear body -->
+    <xacro:property name="HF_height" value="1.560"/> <!-- front body -->
   <xacro:property name="half_wb" value="${B_wheelbase/2.0}"/>
   <xacro:property name="wheel_radius" value="0.80"/>
@@ -24,4 +26,6 @@
   <xacro:property name="box_w" value="${D_width-(2*wheel_width)}"/>
   <xacro:property name="box_h" value="${H_height-F_clearance}"/>
+    <xacro:property name="rbox_h" value="${HR_height-F_clearance}"/>
+    <xacro:property name="fbox_h" value="${HF_height-F_clearance}"/>
     <!-- base footprint -->
     <link name="base_footprint"/>
@@ -54,11 +58,11 @@
     <link name="rear_chassis">
         <visual>
-            <origin xyz="${-rear_box_len/2.0} 0 ${box_h/2.0}"/>
-            <geometry><box size="${rear_box_len} ${box_w} ${box_h}"/></geometry>
+            <origin xyz="${-rear_box_len/2.0} 0 ${rbox_h/2.0}"/>
+            <geometry><box size="${rear_box_len} ${box_w} ${rbox_h}"/></geometry>
             <material name="red"/>
         </visual>
         <collision>
-            <origin xyz="${-rear_box_len/2.0} 0 ${box_h/2.0}"/>
-            <geometry><box size="${rear_box_len} ${box_w} ${box_h}"/></geometry>
+            <origin xyz="${-rear_box_len/2.0} 0 ${rbox_h/2.0}"/>
+            <geometry><box size="${rear_box_len} ${box_w} ${rbox_h}"/></geometry>
         </collision>
         <xacro:box_inertia
@@ -66,6 +70,6 @@
             x="${rear_box_len}"
             y="${box_w}"
-            z="${box_h}"
-            o_xyz="${-rear_box_len/2.0} 0 ${box_h/2.0}"
+            z="${rbox_h}"
+            o_xyz="${-rear_box_len/2.0} 0 ${rbox_h/2.0}"
             o_rpy="0 0 0"/>
     </link>
@@ -73,11 +77,11 @@
     <link name="front_chassis">
         <visual>
-            <origin xyz="${front_box_len/2.0} 0 ${box_h/2.0}"/>
-            <geometry><box size="${front_box_len} ${box_w} ${box_h}"/></geometry>
+            <origin xyz="${front_box_len/2.0} 0 ${fbox_h/2.0}"/>
+            <geometry><box size="${front_box_len} ${box_w} ${fbox_h}"/></geometry>
             <material name="green"/>
         </visual>
         <collision>
-            <origin xyz="${front_box_len/2.0} 0 ${box_h/2.0}"/>
-            <geometry><box size="${front_box_len} ${box_w} ${box_h}"/></geometry>
+            <origin xyz="${front_box_len/2.0} 0 ${fbox_h/2.0}"/>
+            <geometry><box size="${front_box_len} ${box_w} ${fbox_h}"/></geometry>
         </collision>
         <xacro:box_inertia
@@ -85,6 +89,6 @@
             x="${front_box_len}"
             y="${box_w}"
-            z="${box_h}"
-            o_xyz="${front_box_len/2.0} 0 ${box_h/2.0}"
+            z="${fbox_h}"
+            o_xyz="${front_box_len/2.0} 0 ${fbox_h/2.0}"
             o_rpy="0 0 0"/>
     </link>

Commit message: update urdf

File: ros2_ws/src/robot_description/urdf/komatsu.urdf.xacro (robot description, xacro)
@@ -14,18 +14,15 @@
   <xacro:property name="F_clearance" value="0.455"/>
   <xacro:property name="H_height" value="3.395"/>
-  <xacro:property name="X_len" value="2.660"/>
-  <xacro:property name="Y_len" value="2.660"/>
-    <xacro:property name="HR_height" value="2.350"/> <!-- rear body -->
-    <xacro:property name="HF_height" value="1.560"/> <!-- front body -->
+  <xacro:property name="X_len" value="2.660"/> <!-- axes to front and axes to rear -->
   <xacro:property name="half_wb" value="${B_wheelbase/2.0}"/>
   <xacro:property name="wheel_radius" value="0.80"/>
   <xacro:property name="wheel_width" value="0.65"/>
   <xacro:property name="wheel_y" value="${E_track/2.0}"/>
-  <xacro:property name="rear_box_len" value="${Y_len + half_wb}"/>
+  <xacro:property name="rear_box_len" value="${X_len + half_wb}"/>
   <xacro:property name="front_box_len" value="${X_len + half_wb}"/>
   <xacro:property name="box_w" value="${D_width-(2*wheel_width)}"/>
   <xacro:property name="box_h" value="${H_height-F_clearance}"/>
-    <xacro:property name="rbox_h" value="${HR_height-F_clearance}"/>
-    <xacro:property name="fbox_h" value="${HF_height-F_clearance}"/>
+    <xacro:property name="rbox_h" value="${H_height-F_clearance}"/>
+    <xacro:property name="fbox_h" value="${H_height-F_clearance}"/>
     <!-- base footprint -->
     <link name="base_footprint"/>

Commit message: update urdf

File: ros2_ws/src/robot_description/urdf/komatsu.urdf.xacro (robot description, xacro)
@@ -127,5 +127,5 @@
     <parent link="rear_chassis"/>
     <child link="laser_frame"/>
-    <origin xyz="0.0 0.0 ${box_h + 0.03}" rpy="0 0 0"/>
+    <origin xyz="0.0 0.0 ${box_h + 0.3}" rpy="0 0 0"/> <!-- lidar 30 cm above the cabin -->
   </joint>
   <link name="imu_link"/>
