Commit message: increase friction for front wheels

File: ros2_ws/src/robot_description/urdf/fent/fent_gazebo.urdf.xacro (robot description, xacro)
@@ -28,6 +28,6 @@
     <gazebo reference="front_left_wheel">
         <material>Gazebo/Black</material>
-        <mu1>0.05</mu1>
-        <mu2>0.05</mu2>
+        <mu1>0.4</mu1>
+        <mu2>0.4</mu2>
         <kp>1e6</kp>
         <kd>100.0</kd>
@@ -35,6 +35,6 @@
     <gazebo reference="front_right_wheel">
         <material>Gazebo/Black</material>
-        <mu1>0.05</mu1>
-        <mu2>0.05</mu2>
+        <mu1>0.4</mu1>
+        <mu2>0.4</mu2>
         <kp>1e6</kp>
         <kd>100.0</kd>

File: ros2_ws/src/robot_description/urdf/fent/wheels.xacro (robot description, xacro)
@@ -28,4 +28,5 @@
       <origin xyz="${x} ${y} ${z}" rpy="0 0 0"/>
       <axis xyz="0 1 0"/>
+      <dynamics damping="2.0" friction="0.2"/>
     </joint>
   </xacro:macro>
@@ -48,4 +49,5 @@
         <mimic joint="${mimic_joint}" multiplier="${mimic_multiplier}" offset="0.0"/>
       </xacro:if>
+      <dynamics damping="150.0" friction="15.0"/>
     </joint>
     <link name="${name}">
@@ -74,4 +76,5 @@
       <origin xyz="0 0 0" rpy="0 0 0"/>
       <axis xyz="0 1 0"/>
+      <dynamics damping="2.0" friction="0.2"/>
     </joint>
   </xacro:macro>
