Commit message: refactor urdf with single chassis 2

File: ros2_ws/src/robot_description/urdf/fent/fent.urdf.xacro (robot description, xacro)
@@ -46,7 +46,7 @@
     <xacro:property name="weight_r_axle" value="150"/> <!-- x2 -->
     <xacro:property name="total_weight" value="${weight_f_body+weight_r_body+weight_chassis+2*(wheel_weight_f + wheel_weight_r)}"/> <!-- 4300 -->
-    <xacro:property name="chassis_center_z" value="${bottom_clearance + box_height_chassis/2.0 - wheel_rad_rear}"/>
-    <xacro:property name="rear_body_center_z" value="${bottom_clearance + box_height_r_body/2.0 - wheel_rad_rear}"/>
-    <xacro:property name="front_body_center_z" value="${bottom_clearance + box_height_f_body/2.0 - wheel_rad_front}"/>
+    <xacro:property name="chassis_center_z" value="${box_height_chassis/2.0}"/>
+    <xacro:property name="rear_body_center_z" value="${box_height_r_body/2.0}"/>
+    <xacro:property name="front_body_center_z" value="${box_height_f_body/2.0}"/>
     <link name="base_footprint"/>
     <link name="base_link"/>
@@ -54,8 +54,31 @@
         <parent link="base_footprint"/>
         <child link="base_link"/>
-        <origin xyz="0 0 ${wheel_rad_rear}" rpy="0 0 0"/>
+        <origin xyz="0 0 ${bottom_clearance}" rpy="0 0 0"/>
+    </joint>
+    <link name="chassis">
+        <visual>
+            <origin xyz="0 0 ${chassis_center_z}"/>
+            <geometry><box size="${box_len_chassis} ${box_width_chassis} ${box_height_chassis}"/></geometry>
+            <material name="grey"/>
+        </visual>
+        <collision>
+            <origin xyz="0 0 ${chassis_center_z}"/>
+            <geometry><box size="${box_len_chassis} ${box_width_chassis} ${box_height_chassis}"/></geometry>
+        </collision>
+        <xacro:box_inertia
+                m="${weight_chassis}"
+                x="${box_len_chassis}"
+                y="${box_width_chassis}"
+                z="${box_height_chassis}"
+                o_xyz="0 0 ${chassis_center_z}"
+                o_rpy="0 0 0"/>
+    </link>
+    <joint name="base_to_chassis_joint" type="fixed">
+        <parent link="base_link"/>
+        <child link="chassis"/>
+        <origin xyz="0 0 0" rpy="0 0 0"/>
     </joint>
     <joint name="base_to_rear_joint" type="fixed">
-        <parent link="base_link"/>
+        <parent link="chassis"/>
         <child link="rear_body"/>
         <origin xyz="0 0 0" rpy="0 0 0"/>
@@ -98,7 +121,29 @@
     </link>
     <joint name="base_to_front_joint" type="fixed">
-        <parent link="base_link"/>
+        <parent link="chassis"/>
         <child link="front_body"/>
         <origin xyz="0 0 0" rpy="0 0 0"/>
+    </joint>
+    <link name="rear_axle">
+        <visual>
+            <origin xyz="0 0 0" rpy="1.57079632679 0 0"/>
+            <geometry><cylinder radius="${axle_rad_rear}" length="${axle_len_rear}"/></geometry>
+            <material name="grey"/>
+        </visual>
+        <collision>
+            <origin xyz="0 0 0" rpy="1.57079632679 0 0"/>
+            <geometry><cylinder radius="${axle_rad_rear}" length="${axle_len_rear}"/></geometry>
+        </collision>
+        <xacro:cylinder_inertia
+                m="${weight_r_axle}"
+                r="${axle_rad_rear}"
+                l="${axle_len_rear}"
+                o_xyz="0 0 0"
+                o_rpy="0 0 0"/>
+    </link>
+    <joint name="rear_axle_joint" type="fixed">
+        <parent link="chassis"/>
+        <child link="rear_axle"/>
+        <origin xyz="${-half_wheelbase} 0 0" rpy="0 0 0"/>
     </joint>
     <link name="front_axle">
@@ -120,5 +165,5 @@
     </link>
     <joint name="front_axle_roll_joint" type="revolute">
-        <parent link="front_body"/>
+        <parent link="chassis"/>
         <child link="front_axle"/>
         <origin xyz="${half_wheelbase} 0 0" rpy="0 0 0"/>
@@ -127,6 +172,6 @@
     </joint>
     <!-- ===== Wheels ===== -->
-    <xacro:wheel name="rear_left_wheel"  parent="rear_body"  x="${-half_wheelbase}" y="${ wheel_y_distance}" z="0.0" radius="${wheel_rad_rear}" width="${wheel_width_r}" mass="${wheel_weight_r}"/>
-    <xacro:wheel name="rear_right_wheel" parent="rear_body"  x="${-half_wheelbase}" y="${-wheel_y_distance}" z="0.0" radius="${wheel_rad_rear}" width="${wheel_width_r}" mass="${wheel_weight_r}"/>
+    <xacro:wheel name="rear_left_wheel"  parent="rear_axle"  x="0.0" y="${ wheel_y_distance}" z="0.0" radius="${wheel_rad_rear}" width="${wheel_width_r}" mass="${wheel_weight_r}"/>
+    <xacro:wheel name="rear_right_wheel" parent="rear_axle"  x="0.0" y="${-wheel_y_distance}" z="0.0" radius="${wheel_rad_rear}" width="${wheel_width_r}" mass="${wheel_weight_r}"/>
     <xacro:steerable_wheel name="front_left_wheel"  parent="front_axle" x="0.0" y="${ wheel_y_distance}" z="0.0" radius="${wheel_rad_front}" width="${wheel_width_f}" mass="${wheel_weight_f}" steer_limit="${front_steer_limit}"/>
     <xacro:steerable_wheel name="front_right_wheel" parent="front_axle" x="0.0" y="${-wheel_y_distance}" z="0.0" radius="${wheel_rad_front}" width="${wheel_width_f}" mass="${wheel_weight_f}" steer_limit="${front_steer_limit}" mimic_joint="front_left_wheel_steer_joint"/>

Commit message: refactor urdf with single chassis 3

File: ros2_ws/src/robot_description/urdf/fent/fent.urdf.xacro (robot description, xacro)
@@ -46,7 +46,16 @@
     <xacro:property name="weight_r_axle" value="150"/> <!-- x2 -->
     <xacro:property name="total_weight" value="${weight_f_body+weight_r_body+weight_chassis+2*(wheel_weight_f + wheel_weight_r)}"/> <!-- 4300 -->
+    <xacro:property name="base_link_origin_z" value="${bottom_clearance}"/>
     <xacro:property name="chassis_center_z" value="${box_height_chassis/2.0}"/>
-    <xacro:property name="rear_body_center_z" value="${box_height_r_body/2.0}"/>
-    <xacro:property name="front_body_center_z" value="${box_height_f_body/2.0}"/>
+    <xacro:property name="rear_body_origin_x" value="${-box_len_r_body/2.0}"/>
+    <xacro:property name="rear_body_origin_z" value="${box_height_r_body/2.0}"/>
+    <xacro:property name="rear_axle_origin_x" value="${-half_wheelbase}"/>
+    <xacro:property name="rear_axle_origin_z" value="${wheel_rad_rear}"/>
+    <xacro:property name="front_body_origin_x" value="${box_len_f_body/2.0}"/>
+    <xacro:property name="front_body_origin_z" value="${box_height_f_body/2.0}"/>
+    <xacro:property name="front_axle_origin_x" value="${half_wheelbase}"/>
+    <xacro:property name="laser_origin_z" value="${full_height + 0.3}"/>
+    <xacro:property name="gnss_origin_x" value="-1.0"/>
+    <xacro:property name="gnss_origin_z" value="2.0"/>
     <link name="base_footprint"/>
     <link name="base_link"/>
@@ -54,5 +63,5 @@
         <parent link="base_footprint"/>
         <child link="base_link"/>
-        <origin xyz="0 0 ${bottom_clearance}" rpy="0 0 0"/>
+        <origin xyz="0 0 ${base_link_origin_z}" rpy="0 0 0"/>
     </joint>
     <link name="chassis">
@@ -86,10 +95,10 @@
     <link name="rear_body">
         <visual>
-            <origin xyz="${-box_len_r_body/2.0} 0 ${rear_body_center_z}"/>
+            <origin xyz="${rear_body_origin_x} 0 ${rear_body_origin_z}"/>
             <geometry><box size="${box_len_r_body} ${box_width_r_body} ${box_height_r_body}"/></geometry>
             <material name="red"/>
         </visual>
         <collision>
-            <origin xyz="${-box_len_r_body/2.0} 0 ${rear_body_center_z}"/>
+            <origin xyz="${rear_body_origin_x} 0 ${rear_body_origin_z}"/>
             <geometry><box size="${box_len_r_body} ${box_width_r_body} ${box_height_r_body}"/></geometry>
         </collision>
@@ -99,15 +108,15 @@
                 y="${box_width_r_body}"
                 z="${box_height_r_body}"
-                o_xyz="${-box_len_r_body/2.0} 0 ${rear_body_center_z}"
+                o_xyz="${rear_body_origin_x} 0 ${rear_body_origin_z}"
                 o_rpy="0 0 0"/>
     </link>
     <link name="front_body">
         <visual>
-            <origin xyz="${box_len_f_body/2.0} 0 ${front_body_center_z}"/>
+            <origin xyz="${front_body_origin_x} 0 ${front_body_origin_z}"/>
             <geometry><box size="${box_len_f_body} ${box_width_f_body} ${box_height_f_body}"/></geometry>
             <material name="green"/>
         </visual>
         <collision>
-            <origin xyz="${box_len_f_body/2.0} 0 ${front_body_center_z}"/>
+            <origin xyz="${front_body_origin_x} 0 ${front_body_origin_z}"/>
             <geometry><box size="${box_len_f_body} ${box_width_f_body} ${box_height_f_body}"/></geometry>
         </collision>
@@ -117,5 +126,5 @@
                 y="${box_width_f_body}"
                 z="${box_height_f_body}"
-                o_xyz="${box_len_f_body/2.0} 0 ${front_body_center_z}"
+                o_xyz="${front_body_origin_x} 0 ${front_body_origin_z}"
                 o_rpy="0 0 0"/>
     </link>
@@ -145,5 +154,5 @@
         <parent link="chassis"/>
         <child link="rear_axle"/>
-        <origin xyz="${-half_wheelbase} 0 0" rpy="0 0 0"/>
+        <origin xyz="${rear_axle_origin_x} 0 ${rear_axle_origin_z}" rpy="0 0 0"/>
     </joint>
     <link name="front_axle">
@@ -167,5 +176,5 @@
         <parent link="chassis"/>
         <child link="front_axle"/>
-        <origin xyz="${half_wheelbase} 0 0" rpy="0 0 0"/>
+        <origin xyz="${front_axle_origin_x} 0 0" rpy="0 0 0"/>
         <axis xyz="1 0 0"/>
         <limit lower="-0.1745329252" upper="0.1745329252" effort="2000.0" velocity="1.0"/>
@@ -181,5 +190,5 @@
         <parent link="rear_body"/>
         <child link="laser_frame"/>
-        <origin xyz="0.0 0.0 ${full_height + 0.3}" rpy="0 0 0"/>
+        <origin xyz="0.0 0.0 ${laser_origin_z}" rpy="0 0 0"/>
     </joint>
     <link name="imu_link"/>
@@ -193,5 +202,5 @@
         <parent link="base_link"/>
         <child link="gnss_link"/>
-        <origin xyz="-1.0 0.0 2.0" rpy="0 0 0"/>
+        <origin xyz="${gnss_origin_x} 0.0 ${gnss_origin_z}" rpy="0 0 0"/>
     </joint>
 </robot>

Commit message: refactor urdf with single chassis 4

File: ros2_ws/src/robot_description/urdf/fent/fent.urdf.xacro (robot description, xacro)
@@ -25,13 +25,11 @@
     <xacro:property name="axle_rad_rear" value="0.13"/>
     <xacro:property name="axle_len_rear" value="${wheel_track-wheel_width_r}"/>
-    <xacro:property name="axle_to_front_chassis" value="wheel_rad_front"/> <!-- axes to front -->
-    <xacro:property name="axle_to_rear_chassis" value="wheel_rad_front"/> <!-- axes to rear -->
-    <xacro:property name="box_len_chassis" value="${wheelbase + 2*wheel_rad_front}"/>
+    <xacro:property name="box_len_chassis" value="${wheelbase + 2*wheel_rad_front - 0.20}"/>
     <xacro:property name="box_width_chassis" value="0.50"/>
     <xacro:property name="box_height_chassis" value="0.50"/>
     <xacro:property name="axle_to_front_f_body" value="${wheel_rad_front}"/>
     <xacro:property name="box_len_f_body" value="${axle_to_front_f_body + half_wheelbase}"/>
-    <xacro:property name="box_width_f_body" value="0.70"/>
-    <xacro:property name="box_height_f_body" value="1.30"/>
+    <xacro:property name="box_width_f_body" value="0.60"/>
+    <xacro:property name="box_height_f_body" value="0.50"/>
     <xacro:property name="axle_to_r_body" value="0.20"/>
     <xacro:property name="box_len_r_body" value="${axle_to_r_body + half_wheelbase}"/>
@@ -47,15 +45,15 @@
     <xacro:property name="total_weight" value="${weight_f_body+weight_r_body+weight_chassis+2*(wheel_weight_f + wheel_weight_r)}"/> <!-- 4300 -->
     <xacro:property name="base_link_origin_z" value="${bottom_clearance}"/>
-    <xacro:property name="chassis_center_z" value="${box_height_chassis/2.0}"/>
+    <xacro:property name="chassis_origin_z" value="${box_height_chassis/2.0}"/>
+    <xacro:property name="rear_axle_origin_x" value="${-half_wheelbase}"/>
+    <xacro:property name="rear_axle_origin_z" value="${wheel_rad_rear - (bottom_clearance+chassis_origin_z)}"/>
+    <xacro:property name="front_axle_origin_x" value="${half_wheelbase}"/>
+    <xacro:property name="front_axle_origin_z" value="${wheel_rad_front - (bottom_clearance+chassis_origin_z)}"/>
     <xacro:property name="rear_body_origin_x" value="${-box_len_r_body/2.0}"/>
-    <xacro:property name="rear_body_origin_z" value="${box_height_r_body/2.0}"/>
-    <xacro:property name="rear_axle_origin_x" value="${-half_wheelbase}"/>
-    <xacro:property name="rear_axle_origin_z" value="${wheel_rad_rear}"/>
+    <xacro:property name="rear_body_origin_z" value="${box_height_r_body/2.0 - chassis_origin_z}"/>
     <xacro:property name="front_body_origin_x" value="${box_len_f_body/2.0}"/>
-    <xacro:property name="front_body_origin_z" value="${box_height_f_body/2.0}"/>
-    <xacro:property name="front_axle_origin_x" value="${half_wheelbase}"/>
-    <xacro:property name="laser_origin_z" value="${full_height + 0.3}"/>
-    <xacro:property name="gnss_origin_x" value="-1.0"/>
-    <xacro:property name="gnss_origin_z" value="2.0"/>
+    <xacro:property name="front_body_origin_z" value="${box_height_f_body/2.0 + chassis_origin_z}"/>
+    <xacro:property name="laser_origin_z" value="${full_height - bottom_clearance + 0.15}"/>
+    <xacro:property name="gnss_origin_z" value="${full_height - bottom_clearance}"/>
     <link name="base_footprint"/>
     <link name="base_link"/>
@@ -67,10 +65,10 @@
     <link name="chassis">
         <visual>
-            <origin xyz="0 0 ${chassis_center_z}"/>
+            <origin xyz="0 0 0"/>
             <geometry><box size="${box_len_chassis} ${box_width_chassis} ${box_height_chassis}"/></geometry>
             <material name="grey"/>
         </visual>
         <collision>
-            <origin xyz="0 0 ${chassis_center_z}"/>
+            <origin xyz="0 0 0"/>
             <geometry><box size="${box_len_chassis} ${box_width_chassis} ${box_height_chassis}"/></geometry>
         </collision>
@@ -80,5 +78,5 @@
                 y="${box_width_chassis}"
                 z="${box_height_chassis}"
-                o_xyz="0 0 ${chassis_center_z}"
+                o_xyz="0 0 0"
                 o_rpy="0 0 0"/>
     </link>
@@ -86,5 +84,5 @@
         <parent link="base_link"/>
         <child link="chassis"/>
-        <origin xyz="0 0 0" rpy="0 0 0"/>
+        <origin xyz="0 0 ${chassis_origin_z}" rpy="0 0 0"/>
     </joint>
     <joint name="base_to_rear_joint" type="fixed">
@@ -176,5 +174,5 @@
         <parent link="chassis"/>
         <child link="front_axle"/>
-        <origin xyz="${front_axle_origin_x} 0 0" rpy="0 0 0"/>
+        <origin xyz="${front_axle_origin_x} 0 ${front_axle_origin_z}" rpy="0 0 0"/>
         <axis xyz="1 0 0"/>
         <limit lower="-0.1745329252" upper="0.1745329252" effort="2000.0" velocity="1.0"/>
@@ -202,5 +200,5 @@
         <parent link="base_link"/>
         <child link="gnss_link"/>
-        <origin xyz="${gnss_origin_x} 0.0 ${gnss_origin_z}" rpy="0 0 0"/>
+        <origin xyz="0.0 0.0 ${gnss_origin_z}" rpy="0 0 0"/>
     </joint>
 </robot>

File: ros2_ws/src/robot_description/urdf/fent/fent_gazebo.urdf.xacro (robot description, xacro)
@@ -2,13 +2,20 @@
 <robot name="fent" xmlns:xacro="http://www.ros.org/wiki/xacro">
     <xacro:include filename="$(find robot_description)/urdf/fent/fent.urdf.xacro"/>
-    <gazebo reference="rear_chassis">
-        <material>Gazebo/Red</material>
+    <gazebo reference="chassis">
+        <material>Gazebo/DarkGrey</material>
         <mu1>0.5</mu1>
         <mu2>0.5</mu2>
     </gazebo>
-    <gazebo reference="front_chassis">
+    <gazebo reference="front_body">
         <material>Gazebo/Green</material>
-        <mu1>0.5</mu1>
-        <mu2>0.5</mu2>
+    </gazebo>
+    <gazebo reference="rear_body">
+        <material>Gazebo/Red</material>
+    </gazebo>
+    <gazebo reference="rear_axle">
+        <material>Gazebo/DarkGrey</material>
+    </gazebo>
+    <gazebo reference="front_axle">
+        <material>Gazebo/DarkGrey</material>
     </gazebo>
     <gazebo reference="rear_left_wheel">
@@ -94,6 +101,6 @@
             <left_joint>rear_left_wheel_joint</left_joint>
             <right_joint>rear_right_wheel_joint</right_joint>
-            <wheel_separation>${E_track}</wheel_separation>
-            <wheel_diameter>${2.0 * wheel_rad_r}</wheel_diameter>
+            <wheel_separation>${wheel_track}</wheel_separation>
+            <wheel_diameter>${2.0 * wheel_rad_rear}</wheel_diameter>
             <max_wheel_torque>80000</max_wheel_torque>
             <max_wheel_acceleration>20.0</max_wheel_acceleration>
