Commit message: set P12 for gz 5

File: ros2_ws/src/robot_description/urdf/komatsu/komatsu_gazebo.urdf.xacro (robot description, xacro)
@@ -93,37 +93,51 @@
         </sensor>
     </gazebo>
-    <!-- ===== Differential Drive Plugin for Simplified Motion ===== -->
-    <!-- This plugin provides a simple differential drive interface for cmd_vel -->
+    <!-- ros2_control interfaces for articulated drive in Gazebo -->
+    <ros2_control name="KomatsuGazeboSystem" type="system">
+        <hardware>
+            <plugin>gazebo_ros2_control/GazeboSystem</plugin>
+        </hardware>
+        <joint name="rear_left_wheel_joint">
+            <command_interface name="velocity"/>
+            <state_interface name="position"/>
+            <state_interface name="velocity"/>
+        </joint>
+        <joint name="rear_right_wheel_joint">
+            <command_interface name="velocity"/>
+            <state_interface name="position"/>
+            <state_interface name="velocity"/>
+        </joint>
+        <joint name="front_left_wheel_joint">
+            <command_interface name="velocity"/>
+            <state_interface name="position"/>
+            <state_interface name="velocity"/>
+        </joint>
+        <joint name="front_right_wheel_joint">
+            <command_interface name="velocity"/>
+            <state_interface name="position"/>
+            <state_interface name="velocity"/>
+        </joint>
+        <joint name="articulation_to_front">
+            <command_interface name="position"/>
+            <state_interface name="position"/>
+            <state_interface name="velocity"/>
+        </joint>
+    </ros2_control>
     <gazebo>
-        <plugin name="differential_drive_controller" filename="libgazebo_ros_diff_drive.so">
+        <plugin name="gazebo_ros2_control" filename="libgazebo_ros2_control.so">
+            <parameters>$(find robot_bringup)/config/komatsu_ros2_controllers.yaml</parameters>
+        </plugin>
+    </gazebo>
+    <gazebo>
+        <plugin name="gazebo_ros_p3d" filename="libgazebo_ros_p3d.so">
             <ros>
                 <namespace>/</namespace>
-                <remapping>/cmd_vel:=/cmd_vel_ll</remapping>
+                <remapping>odom:=/odom</remapping>
             </ros>
-            <!-- Wheels -->
-            <left_joint>rear_left_wheel_joint</left_joint>
-            <right_joint>rear_right_wheel_joint</right_joint>
-            <!-- Kinematics -->
-            <wheel_separation>2.160</wheel_separation>
-            <wheel_diameter>1.6</wheel_diameter>
-            <!-- Limits -->
-            <max_wheel_torque>120000</max_wheel_torque>
-            <max_wheel_acceleration>35.0</max_wheel_acceleration>
-            <!-- Output -->
-            <publish_odom>true</publish_odom>
-            <publish_odom_tf>false</publish_odom_tf>
-            <publish_wheel_tf>false</publish_wheel_tf>
-            <!-- Keep /odom consistent with Gazebo world pose to match GNSS motion. -->
-            <odometrySource>world</odometrySource>
-            <odometry_frame>odom</odometry_frame>
-            <robot_base_frame>base_footprint</robot_base_frame>
-            <!-- Topics -->
-            <command_topic>cmd_vel_ll</command_topic>
-            <odometry_topic>odom</odometry_topic>
-            <!-- Update rate -->
+            <body_name>base_footprint</body_name>
             <update_rate>50.0</update_rate>
+            <gaussian_noise>0.0</gaussian_noise>
         </plugin>
     </gazebo>
-    <!-- Ground-truth p3d plugin removed from default bringup to avoid invalid-link errors. -->
     <!-- ===== GPS / NavSat Plugin ===== -->
     <gazebo reference="gnss_link">
@@ -139,17 +153,3 @@
         </sensor>
     </gazebo>
-    <!-- ===== Joint State Publisher Plugin ===== -->
-    <gazebo>
-        <plugin name="joint_state_publisher" filename="libgazebo_ros_joint_state_publisher.so">
-            <ros>
-                <namespace>/</namespace>
-            </ros>
-            <update_rate>50.0</update_rate>
-            <joint_name>rear_left_wheel_joint</joint_name>
-            <joint_name>rear_right_wheel_joint</joint_name>
-            <joint_name>front_left_wheel_joint</joint_name>
-            <joint_name>front_right_wheel_joint</joint_name>
-            <joint_name>articulation_to_front</joint_name>
-        </plugin>
-    </gazebo>
 </robot>

File: ros2_ws/src/robot_description/urdf/komatsu/wheels.xacro (robot description, xacro)
@@ -41,4 +41,6 @@
       <!-- wheel rolls around Y (left axis), with ROS convention x forward, y left, z up -->
       <axis xyz="0 1 0"/>
+      <limit effort="300000" velocity="25.0"/>
+      <dynamics damping="0.5" friction="0.01"/>
     </joint>
   </xacro:macro>
