Commit message: set P12 for gz

File: ros2_ws/src/robot_description/urdf/komatsu/komatsu.urdf.xacro (robot description, xacro)
@@ -86,9 +86,12 @@
                 o_rpy="0 0 0"/>
     </link>
-    <!-- articulation joints - temporarily fixed for stability -->
-    <joint name="articulation_to_front" type="fixed">
+    <!-- Simplified articulation: rear body is fixed to the articulation center, front yaws around it. -->
+    <joint name="articulation_to_front" type="revolute">
         <parent link="articulation_link"/>
         <child link="front_chassis"/>
         <origin xyz="0 0 0" rpy="0 0 0"/>
+        <axis xyz="0 0 1"/>
+        <limit lower="-0.610865" upper="0.610865" effort="80000" velocity="1.2"/>
+        <dynamics damping="120.0" friction="8.0"/>
     </joint>
     <joint name="articulation_to_rear" type="fixed">

File: ros2_ws/src/robot_description/urdf/komatsu/komatsu_gazebo.urdf.xacro (robot description, xacro)
@@ -19,5 +19,5 @@
         <mu1>1.0</mu1>
         <mu2>1.0</mu2>
-        <kp>1e6</kp>
+        <kp>4e6</kp>
         <kd>100.0</kd>
     </gazebo>
@@ -26,19 +26,19 @@
         <mu1>1.0</mu1>
         <mu2>1.0</mu2>
-        <kp>1e6</kp>
+        <kp>4e6</kp>
         <kd>100.0</kd>
     </gazebo>
     <gazebo reference="front_left_wheel">
         <material>Gazebo/Black</material>
-        <mu1>0.05</mu1>
-        <mu2>0.05</mu2>
-        <kp>1e6</kp>
+        <mu1>1.0</mu1>
+        <mu2>1.0</mu2>
+        <kp>4e6</kp>
         <kd>100.0</kd>
     </gazebo>
     <gazebo reference="front_right_wheel">
         <material>Gazebo/Black</material>
-        <mu1>0.05</mu1>
-        <mu2>0.05</mu2>
-        <kp>1e6</kp>
+        <mu1>1.0</mu1>
+        <mu2>1.0</mu2>
+        <kp>4e6</kp>
         <kd>100.0</kd>
     </gazebo>
@@ -99,4 +99,5 @@
             <ros>
                 <namespace>/</namespace>
+                <remapping>/cmd_vel:=/cmd_vel_ll</remapping>
             </ros>
             <!-- Wheels -->
@@ -104,22 +105,22 @@
             <right_joint>rear_right_wheel_joint</right_joint>
             <!-- Kinematics -->
-            <wheel_separation>2.160</wheel_separation>
-            <wheel_diameter>1.6</wheel_diameter>
+            <wheelSeparation>2.160</wheelSeparation>
+            <wheelDiameter>1.6</wheelDiameter>
             <!-- Limits -->
             <max_wheel_torque>80000</max_wheel_torque>
             <max_wheel_acceleration>20.0</max_wheel_acceleration>
             <!-- Output -->
-            <publish_odom>true</publish_odom>
-            <publish_odom_tf>false</publish_odom_tf>
-            <publish_wheel_tf>false</publish_wheel_tf>
+            <publishOdom>true</publishOdom>
+            <publishOdomTF>false</publishOdomTF>
+            <publishWheelTF>false</publishWheelTF>
             <!-- Keep /odom consistent with Gazebo world pose to match GNSS motion. -->
             <odometrySource>world</odometrySource>
-            <odometry_frame>odom</odometry_frame>
-            <robot_base_frame>base_footprint</robot_base_frame>
+            <odometryFrame>odom</odometryFrame>
+            <robotBaseFrame>base_footprint</robotBaseFrame>
             <!-- Topics -->
-            <command_topic>cmd_vel</command_topic>
-            <odometry_topic>odom</odometry_topic>
+            <commandTopic>cmd_vel_ll</commandTopic>
+            <odometryTopic>odom</odometryTopic>
             <!-- Update rate -->
-            <update_rate>50.0</update_rate>
+            <updateRate>50.0</updateRate>
         </plugin>
     </gazebo>
@@ -149,4 +150,5 @@
             <joint_name>front_left_wheel_joint</joint_name>
             <joint_name>front_right_wheel_joint</joint_name>
+            <joint_name>articulation_to_front</joint_name>
         </plugin>
     </gazebo>

Commit message: set P12 for gz 2

File: ros2_ws/src/robot_description/urdf/komatsu/komatsu.urdf.xacro (robot description, xacro)
@@ -48,4 +48,6 @@
     <xacro:property name="body_center_z" value="${F_clearance + box_h/2.0 - wheel_radius}"/>
     <xacro:property name="body_top_z" value="${body_center_z + box_h/2.0}"/>
+    <!-- Lower COM than geometric center to better approximate wheel-loader mass distribution. -->
+    <xacro:property name="body_com_z" value="${body_center_z - 0.65}"/>
     <!-- rear body -->
     <link name="rear_chassis">
@@ -60,9 +62,9 @@
         </collision>
         <xacro:box_inertia
-                m="500.0"
+                m="9000.0"
                 x="${rear_box_len}"
                 y="${box_w}"
                 z="${box_h}"
-                o_xyz="${-rear_box_len/2.0} 0 ${body_center_z}"
+                o_xyz="${-rear_box_len/2.0} 0 ${body_com_z}"
                 o_rpy="0 0 0"/>
     </link>
@@ -79,9 +81,9 @@
         </collision>
         <xacro:box_inertia
-                m="500.0"
+                m="9000.0"
                 x="${front_box_len}"
                 y="${box_w}"
                 z="${box_h}"
-                o_xyz="${front_box_len/2.0} 0 ${body_center_z}"
+                o_xyz="${front_box_len/2.0} 0 ${body_com_z}"
                 o_rpy="0 0 0"/>
     </link>
@@ -92,6 +94,6 @@
         <origin xyz="0 0 0" rpy="0 0 0"/>
         <axis xyz="0 0 1"/>
-        <limit lower="-0.610865" upper="0.610865" effort="80000" velocity="1.2"/>
-        <dynamics damping="120.0" friction="8.0"/>
+        <limit lower="-0.558505" upper="0.558505" effort="120000" velocity="0.35"/>
+        <dynamics damping="320.0" friction="35.0"/>
     </joint>
     <joint name="articulation_to_rear" type="fixed">

File: ros2_ws/src/robot_description/urdf/komatsu/komatsu_gazebo.urdf.xacro (robot description, xacro)
@@ -105,22 +105,22 @@
             <right_joint>rear_right_wheel_joint</right_joint>
             <!-- Kinematics -->
-            <wheelSeparation>2.160</wheelSeparation>
-            <wheelDiameter>1.6</wheelDiameter>
+            <wheel_separation>2.160</wheel_separation>
+            <wheel_diameter>1.6</wheel_diameter>
             <!-- Limits -->
             <max_wheel_torque>80000</max_wheel_torque>
             <max_wheel_acceleration>20.0</max_wheel_acceleration>
             <!-- Output -->
-            <publishOdom>true</publishOdom>
-            <publishOdomTF>false</publishOdomTF>
-            <publishWheelTF>false</publishWheelTF>
+            <publish_odom>true</publish_odom>
+            <publish_odom_tf>false</publish_odom_tf>
+            <publish_wheel_tf>false</publish_wheel_tf>
             <!-- Keep /odom consistent with Gazebo world pose to match GNSS motion. -->
             <odometrySource>world</odometrySource>
-            <odometryFrame>odom</odometryFrame>
-            <robotBaseFrame>base_footprint</robotBaseFrame>
+            <odometry_frame>odom</odometry_frame>
+            <robot_base_frame>base_footprint</robot_base_frame>
             <!-- Topics -->
-            <commandTopic>cmd_vel_ll</commandTopic>
-            <odometryTopic>odom</odometryTopic>
+            <command_topic>cmd_vel_ll</command_topic>
+            <odometry_topic>odom</odometry_topic>
             <!-- Update rate -->
-            <updateRate>50.0</updateRate>
+            <update_rate>50.0</update_rate>
         </plugin>
     </gazebo>

Commit message: set P12 for gz 3

File: ros2_ws/src/robot_description/urdf/komatsu/komatsu.urdf.xacro (robot description, xacro)
@@ -48,6 +48,6 @@
     <xacro:property name="body_center_z" value="${F_clearance + box_h/2.0 - wheel_radius}"/>
     <xacro:property name="body_top_z" value="${body_center_z + box_h/2.0}"/>
-    <!-- Lower COM than geometric center to better approximate wheel-loader mass distribution. -->
-    <xacro:property name="body_com_z" value="${body_center_z - 0.65}"/>
+    <!-- Keep COM lower than geometric center, but not extreme for simplified Gazebo dynamics. -->
+    <xacro:property name="body_com_z" value="${body_center_z - 0.25}"/>
     <!-- rear body -->
     <link name="rear_chassis">
@@ -62,5 +62,5 @@
         </collision>
         <xacro:box_inertia
-                m="9000.0"
+                m="2500.0"
                 x="${rear_box_len}"
                 y="${box_w}"
@@ -81,5 +81,5 @@
         </collision>
         <xacro:box_inertia
-                m="9000.0"
+                m="2500.0"
                 x="${front_box_len}"
                 y="${box_w}"
@@ -94,6 +94,6 @@
         <origin xyz="0 0 0" rpy="0 0 0"/>
         <axis xyz="0 0 1"/>
-        <limit lower="-0.558505" upper="0.558505" effort="120000" velocity="0.35"/>
-        <dynamics damping="320.0" friction="35.0"/>
+        <limit lower="-0.558505" upper="0.558505" effort="80000" velocity="0.8"/>
+        <dynamics damping="80.0" friction="5.0"/>
     </joint>
     <joint name="articulation_to_rear" type="fixed">

File: ros2_ws/src/robot_description/urdf/komatsu/komatsu_gazebo.urdf.xacro (robot description, xacro)
@@ -17,29 +17,29 @@
     <gazebo reference="rear_left_wheel">
         <material>Gazebo/Black</material>
-        <mu1>1.0</mu1>
-        <mu2>1.0</mu2>
-        <kp>4e6</kp>
-        <kd>100.0</kd>
+        <mu1>0.6</mu1>
+        <mu2>0.6</mu2>
+        <kp>1e5</kp>
+        <kd>10.0</kd>
     </gazebo>
     <gazebo reference="rear_right_wheel">
         <material>Gazebo/Black</material>
-        <mu1>1.0</mu1>
-        <mu2>1.0</mu2>
-        <kp>4e6</kp>
-        <kd>100.0</kd>
+        <mu1>0.6</mu1>
+        <mu2>0.6</mu2>
+        <kp>1e5</kp>
+        <kd>10.0</kd>
     </gazebo>
     <gazebo reference="front_left_wheel">
         <material>Gazebo/Black</material>
-        <mu1>1.0</mu1>
-        <mu2>1.0</mu2>
-        <kp>4e6</kp>
-        <kd>100.0</kd>
+        <mu1>0.6</mu1>
+        <mu2>0.6</mu2>
+        <kp>1e5</kp>
+        <kd>10.0</kd>
     </gazebo>
     <gazebo reference="front_right_wheel">
         <material>Gazebo/Black</material>
-        <mu1>1.0</mu1>
-        <mu2>1.0</mu2>
-        <kp>4e6</kp>
-        <kd>100.0</kd>
+        <mu1>0.6</mu1>
+        <mu2>0.6</mu2>
+        <kp>1e5</kp>
+        <kd>10.0</kd>
     </gazebo>
     <!-- ===== Sensors ===== -->
@@ -108,6 +108,6 @@
             <wheel_diameter>1.6</wheel_diameter>
             <!-- Limits -->
-            <max_wheel_torque>80000</max_wheel_torque>
-            <max_wheel_acceleration>20.0</max_wheel_acceleration>
+            <max_wheel_torque>120000</max_wheel_torque>
+            <max_wheel_acceleration>35.0</max_wheel_acceleration>
             <!-- Output -->
             <publish_odom>true</publish_odom>

Commit message: adjust, mu, kp, kd

File: ros2_ws/src/robot_description/urdf/komatsu/komatsu.urdf.xacro (robot description, xacro)
@@ -23,4 +23,9 @@
     <xacro:property name="box_w" value="${D_width-(2*wheel_width)}"/>
     <xacro:property name="box_h" value="${H_height-F_clearance}"/>
+    <!-- Dynamics tuning for a heavier articulated loader body model -->
+    <xacro:property name="rear_chassis_mass" value="8500.0"/>
+    <xacro:property name="front_chassis_mass" value="8500.0"/>
+    <xacro:property name="articulation_damping" value="650.0"/>
+    <xacro:property name="articulation_friction" value="45.0"/>
     <!-- Ground frame -->
     <link name="base_footprint"/>
@@ -48,6 +53,6 @@
     <xacro:property name="body_center_z" value="${F_clearance + box_h/2.0 - wheel_radius}"/>
     <xacro:property name="body_top_z" value="${body_center_z + box_h/2.0}"/>
-    <!-- Keep COM lower than geometric center, but not extreme for simplified Gazebo dynamics. -->
-    <xacro:property name="body_com_z" value="${body_center_z - 0.25}"/>
+    <!-- Place COM at the bottom quarter of body height (bottom + box_h/4). -->
+    <xacro:property name="body_com_z" value="${body_center_z - box_h/4.0}"/>
     <!-- rear body -->
     <link name="rear_chassis">
@@ -62,5 +67,5 @@
         </collision>
         <xacro:box_inertia
-                m="2500.0"
+                m="${rear_chassis_mass}"
                 x="${rear_box_len}"
                 y="${box_w}"
@@ -81,5 +86,5 @@
         </collision>
         <xacro:box_inertia
-                m="2500.0"
+                m="${front_chassis_mass}"
                 x="${front_box_len}"
                 y="${box_w}"
@@ -95,5 +100,5 @@
         <axis xyz="0 0 1"/>
         <limit lower="-0.558505" upper="0.558505" effort="80000" velocity="0.8"/>
-        <dynamics damping="80.0" friction="5.0"/>
+        <dynamics damping="${articulation_damping}" friction="${articulation_friction}"/>
     </joint>
     <joint name="articulation_to_rear" type="fixed">

File: ros2_ws/src/robot_description/urdf/komatsu/komatsu_gazebo.urdf.xacro (robot description, xacro)
@@ -3,43 +3,73 @@
     <!-- Include base robot model -->
     <xacro:include filename="$(find robot_description)/urdf/komatsu/komatsu.urdf.xacro"/>
+    <!-- Contact and joint tuning for Gazebo classic -->
+    <xacro:property name="wheel_mu" value="1.15"/>
+    <xacro:property name="wheel_kp" value="2500000.0"/>
+    <xacro:property name="wheel_kd" value="22000.0"/>
+    <xacro:property name="wheel_min_depth" value="0.004"/>
+    <xacro:property name="wheel_max_vel" value="0.25"/>
+    <xacro:property name="wheel_slip" value="0.015"/>
+    <xacro:property name="articulation_spring_k" value="2500.0"/>
+    <xacro:property name="articulation_spring_ref" value="0.0"/>
     <!-- ===== Gazebo Material Properties ===== -->
     <gazebo reference="rear_chassis">
         <material>Gazebo/Red</material>
-        <mu1>0.5</mu1>
-        <mu2>0.5</mu2>
+        <mu1>0.7</mu1>
+        <mu2>0.7</mu2>
     </gazebo>
     <gazebo reference="front_chassis">
         <material>Gazebo/Green</material>
-        <mu1>0.5</mu1>
-        <mu2>0.5</mu2>
+        <mu1>0.7</mu1>
+        <mu2>0.7</mu2>
     </gazebo>
     <!-- Wheel friction properties -->
     <gazebo reference="rear_left_wheel">
         <material>Gazebo/Black</material>
-        <mu1>0.6</mu1>
-        <mu2>0.6</mu2>
-        <kp>1e5</kp>
-        <kd>10.0</kd>
+        <mu1>${wheel_mu}</mu1>
+        <mu2>${wheel_mu}</mu2>
+        <kp>${wheel_kp}</kp>
+        <kd>${wheel_kd}</kd>
+        <minDepth>${wheel_min_depth}</minDepth>
+        <maxVel>${wheel_max_vel}</maxVel>
+        <slip1>${wheel_slip}</slip1>
+        <slip2>${wheel_slip}</slip2>
     </gazebo>
     <gazebo reference="rear_right_wheel">
         <material>Gazebo/Black</material>
-        <mu1>0.6</mu1>
-        <mu2>0.6</mu2>
-        <kp>1e5</kp>
-        <kd>10.0</kd>
+        <mu1>${wheel_mu}</mu1>
+        <mu2>${wheel_mu}</mu2>
+        <kp>${wheel_kp}</kp>
+        <kd>${wheel_kd}</kd>
+        <minDepth>${wheel_min_depth}</minDepth>
+        <maxVel>${wheel_max_vel}</maxVel>
+        <slip1>${wheel_slip}</slip1>
+        <slip2>${wheel_slip}</slip2>
     </gazebo>
     <gazebo reference="front_left_wheel">
         <material>Gazebo/Black</material>
-        <mu1>0.6</mu1>
-        <mu2>0.6</mu2>
-        <kp>1e5</kp>
-        <kd>10.0</kd>
+        <mu1>${wheel_mu}</mu1>
+        <mu2>${wheel_mu}</mu2>
+        <kp>${wheel_kp}</kp>
+        <kd>${wheel_kd}</kd>
+        <minDepth>${wheel_min_depth}</minDepth>
+        <maxVel>${wheel_max_vel}</maxVel>
+        <slip1>${wheel_slip}</slip1>
+        <slip2>${wheel_slip}</slip2>
     </gazebo>
     <gazebo reference="front_right_wheel">
         <material>Gazebo/Black</material>
-        <mu1>0.6</mu1>
-        <mu2>0.6</mu2>
-        <kp>1e5</kp>
-        <kd>10.0</kd>
+        <mu1>${wheel_mu}</mu1>
+        <mu2>${wheel_mu}</mu2>
+        <kp>${wheel_kp}</kp>
+        <kd>${wheel_kd}</kd>
+        <minDepth>${wheel_min_depth}</minDepth>
+        <maxVel>${wheel_max_vel}</maxVel>
+        <slip1>${wheel_slip}</slip1>
+        <slip2>${wheel_slip}</slip2>
+    </gazebo>
+    <gazebo reference="articulation_to_front">
+        <implicitSpringDamper>true</implicitSpringDamper>
+        <springStiffness>${articulation_spring_k}</springStiffness>
+        <springReference>${articulation_spring_ref}</springReference>
     </gazebo>
     <!-- ===== Sensors ===== -->
