Commit message: fix drift issue

File: ros2_ws/src/robot_description/urdf/fendt/fendt_gazebo.urdf.xacro (robot description, xacro)
@@ -9,6 +9,6 @@
         <mu2>0.5</mu2>
         <velocity_decay>
-            <linear>0.2</linear>
-            <angular>0.2</angular>
+            <linear>0.0</linear>
+            <angular>0.0</angular>
         </velocity_decay>
     </gazebo>
@@ -51,37 +51,37 @@
     <gazebo reference="rear_left_wheel">
         <material>Gazebo/Black</material>
-        <mu1>3.2</mu1>
-        <mu2>3.2</mu2>
-        <kp>1e7</kp>
-        <kd>1000.0</kd>
-        <slip1>0.0</slip1>
-        <slip2>0.0</slip2>
+        <mu1>2.2</mu1>
+        <mu2>2.2</mu2>
+        <kp>1e7</kp>
+        <kd>1000.0</kd>
+        <slip1>0.02</slip1>
+        <slip2>0.02</slip2>
     </gazebo>
     <gazebo reference="rear_right_wheel">
         <material>Gazebo/Black</material>
-        <mu1>3.2</mu1>
-        <mu2>3.2</mu2>
-        <kp>1e7</kp>
-        <kd>1000.0</kd>
-        <slip1>0.0</slip1>
-        <slip2>0.0</slip2>
+        <mu1>2.2</mu1>
+        <mu2>2.2</mu2>
+        <kp>1e7</kp>
+        <kd>1000.0</kd>
+        <slip1>0.02</slip1>
+        <slip2>0.02</slip2>
     </gazebo>
     <gazebo reference="front_left_wheel">
         <material>Gazebo/Black</material>
-        <mu1>3.2</mu1>
-        <mu2>3.2</mu2>
-        <kp>1e7</kp>
-        <kd>1000.0</kd>
-        <slip1>0.0</slip1>
-        <slip2>0.0</slip2>
+        <mu1>2.2</mu1>
+        <mu2>2.2</mu2>
+        <kp>1e7</kp>
+        <kd>1000.0</kd>
+        <slip1>0.02</slip1>
+        <slip2>0.02</slip2>
     </gazebo>
     <gazebo reference="front_right_wheel">
         <material>Gazebo/Black</material>
-        <mu1>3.2</mu1>
-        <mu2>3.2</mu2>
-        <kp>1e7</kp>
-        <kd>1000.0</kd>
-        <slip1>0.0</slip1>
-        <slip2>0.0</slip2>
+        <mu1>2.2</mu1>
+        <mu2>2.2</mu2>
+        <kp>1e7</kp>
+        <kd>1000.0</kd>
+        <slip1>0.02</slip1>
+        <slip2>0.02</slip2>
     </gazebo>
     <gazebo reference="laser_frame">

File: ros2_ws/src/robot_description/urdf/fendt/wheels.xacro (robot description, xacro)
@@ -56,5 +56,5 @@
       <origin xyz="0 ${pivot_y_offset} 0" rpy="0 0 0"/>
       <axis xyz="0 1 0"/>
-      <dynamics damping="25.0" friction="6.0"/>
+      <dynamics damping="3.0" friction="0.4"/>
     </joint>
     <link name="${name}">
@@ -117,5 +117,5 @@
         <mimic joint="${mimic_joint}" multiplier="${mimic_multiplier}" offset="0.0"/>
       </xacro:if>
-      <dynamics damping="300.0" friction="45.0"/>
+      <dynamics damping="70.0" friction="5.0"/>
     </joint>
     <link name="${name}_hub">
@@ -144,5 +144,5 @@
       <origin xyz="0 ${pivot_y_offset} 0" rpy="0 0 0"/>
       <axis xyz="0 1 0"/>
-      <dynamics damping="20.0" friction="5.0"/>
+      <dynamics damping="2.8" friction="0.35"/>
     </joint>
     <link name="${name}">
