Commit message: ros2 controller pkg

File: ros2_ws/src/robot_description/urdf/fendt/fendt.urdf.xacro (robot description, xacro)
@@ -182,5 +182,5 @@
     <xacro:wheel name="rear_right_wheel" parent="rear_axle"  x="0.0" y="${-wheel_y_distance}" z="0.0" radius="${wheel_rad_rear}" width="${wheel_width_r}" mass="${wheel_weight_r}"/>
     <xacro:steerable_wheel name="front_left_wheel"  parent="front_axle" x="0.0" y="${ wheel_y_distance}" z="0.0" radius="${wheel_rad_front}" width="${wheel_width_f}" mass="${wheel_weight_f}" steer_limit="${front_steer_limit}"/>
-    <xacro:steerable_wheel name="front_right_wheel" parent="front_axle" x="0.0" y="${-wheel_y_distance}" z="0.0" radius="${wheel_rad_front}" width="${wheel_width_f}" mass="${wheel_weight_f}" steer_limit="${front_steer_limit}" mimic_joint="front_left_wheel_steer_joint"/>
+    <xacro:steerable_wheel name="front_right_wheel" parent="front_axle" x="0.0" y="${-wheel_y_distance}" z="0.0" radius="${wheel_rad_front}" width="${wheel_width_f}" mass="${wheel_weight_f}" steer_limit="${front_steer_limit}"/>
     <!-- ===== Sensors ===== -->
     <link name="laser_frame"/>

File: ros2_ws/src/robot_description/urdf/fendt/fendt_gazebo.urdf.xacro (robot description, xacro)
@@ -37,6 +37,6 @@
     <gazebo reference="front_left_wheel">
         <material>Gazebo/Black</material>
-        <mu1>0.04</mu1>
-        <mu2>0.04</mu2>
+        <mu1>1.0</mu1>
+        <mu2>1.0</mu2>
         <kp>4e6</kp>
         <kd>100.0</kd>
@@ -44,6 +44,6 @@
     <gazebo reference="front_right_wheel">
         <material>Gazebo/Black</material>
-        <mu1>0.04</mu1>
-        <mu2>0.04</mu2>
+        <mu1>1.0</mu1>
+        <mu2>1.0</mu2>
         <kp>4e6</kp>
         <kd>100.0</kd>

File: ros2_ws/src/robot_description/urdf/fendt/wheels.xacro (robot description, xacro)
@@ -40,5 +40,5 @@
       </inertial>
     </link>
-    <joint name="${name}_steer_joint" type="fixed">
+    <joint name="${name}_steer_joint" type="revolute">
       <parent link="${parent}"/>
       <child link="${name}_steer"/>

Commit message: NAV2 GOAL REACHED, ackermann steering ros2 control

File: ros2_ws/src/robot_description/urdf/fendt/fendt.urdf.xacro (robot description, xacro)
@@ -171,10 +171,8 @@
                 o_rpy="0 0 0"/>
     </link>
-    <joint name="front_axle_roll_joint" type="revolute">
+    <joint name="front_axle_roll_joint" type="fixed">
         <parent link="chassis"/>
         <child link="front_axle"/>
         <origin xyz="${front_axle_origin_x} 0 ${front_axle_origin_z}" rpy="0 0 0"/>
-        <axis xyz="1 0 0"/>
-        <limit lower="-0.1745329252" upper="0.1745329252" effort="2000.0" velocity="1.0"/>
     </joint>
     <!-- ===== Wheels ===== -->

Commit message: fix physic issues

File: ros2_ws/src/robot_description/urdf/fendt/fendt.urdf.xacro (robot description, xacro)
@@ -102,5 +102,5 @@
         </collision>
         <xacro:box_inertia
-                m="${weight_f_body}"
+                m="${weight_r_body}"
                 x="${box_len_r_body}"
                 y="${box_width_r_body}"

File: ros2_ws/src/robot_description/urdf/fendt/wheels.xacro (robot description, xacro)
@@ -28,5 +28,5 @@
       <origin xyz="${x} ${y} ${z}" rpy="0 0 0"/>
       <axis xyz="0 1 0"/>
-      <dynamics damping="2.0" friction="0.2"/>
+      <dynamics damping="12.0" friction="2.0"/>
     </joint>
   </xacro:macro>
@@ -76,5 +76,5 @@
       <origin xyz="0 0 0" rpy="0 0 0"/>
       <axis xyz="0 1 0"/>
-      <dynamics damping="2.0" friction="0.2"/>
+      <dynamics damping="10.0" friction="1.5"/>
     </joint>
   </xacro:macro>

Commit message: fix physic issues 2

File: ros2_ws/src/robot_description/urdf/fendt/fendt.urdf.xacro (robot description, xacro)
@@ -36,6 +36,6 @@
     <xacro:property name="box_width_r_body" value="${full_width-(2*wheel_width_r)}"/>
     <xacro:property name="box_height_r_body" value="${full_height-bottom_clearance}"/>
-    <xacro:property name="weight_f_body" value="50"/>
-    <xacro:property name="weight_r_body" value="500"/>
+    <xacro:property name="weight_f_body" value="150"/>
+    <xacro:property name="weight_r_body" value="250"/>
     <xacro:property name="weight_chassis" value="3000"/>
     <xacro:property name="wheel_weight_f" value="100"/> <!-- x2 -->

File: ros2_ws/src/robot_description/urdf/fendt/fendt_gazebo.urdf.xacro (robot description, xacro)
@@ -23,29 +23,29 @@
     <gazebo reference="rear_left_wheel">
         <material>Gazebo/Black</material>
-        <mu1>1.0</mu1>
-        <mu2>1.0</mu2>
-        <kp>4e6</kp>
-        <kd>100.0</kd>
+        <mu1>2.5</mu1>
+        <mu2>2.5</mu2>
+        <kp>1e7</kp>
+        <kd>500.0</kd>
     </gazebo>
     <gazebo reference="rear_right_wheel">
         <material>Gazebo/Black</material>
-        <mu1>1.0</mu1>
-        <mu2>1.0</mu2>
-        <kp>4e6</kp>
-        <kd>100.0</kd>
+        <mu1>2.5</mu1>
+        <mu2>2.5</mu2>
+        <kp>1e7</kp>
+        <kd>500.0</kd>
     </gazebo>
     <gazebo reference="front_left_wheel">
         <material>Gazebo/Black</material>
-        <mu1>1.0</mu1>
-        <mu2>1.0</mu2>
-        <kp>4e6</kp>
-        <kd>100.0</kd>
+        <mu1>2.5</mu1>
+        <mu2>2.5</mu2>
+        <kp>1e7</kp>
+        <kd>500.0</kd>
     </gazebo>
     <gazebo reference="front_right_wheel">
         <material>Gazebo/Black</material>
-        <mu1>1.0</mu1>
-        <mu2>1.0</mu2>
-        <kp>4e6</kp>
-        <kd>100.0</kd>
+        <mu1>2.5</mu1>
+        <mu2>2.5</mu2>
+        <kp>1e7</kp>
+        <kd>500.0</kd>
     </gazebo>
     <gazebo reference="laser_frame">
@@ -100,4 +100,42 @@
             <always_on>true</always_on>
             <update_rate>10</update_rate>
+            <gps>
+                <position_sensing>
+                    <horizontal>
+                        <noise type="gaussian">
+                            <mean>0.0</mean>
+                            <stddev>0.02</stddev>
+                            <bias_mean>0.0</bias_mean>
+                            <bias_stddev>0.0</bias_stddev>
+                        </noise>
+                    </horizontal>
+                    <vertical>
+                        <noise type="gaussian">
+                            <mean>0.0</mean>
+                            <stddev>0.03</stddev>
+                            <bias_mean>0.0</bias_mean>
+                            <bias_stddev>0.0</bias_stddev>
+                        </noise>
+                    </vertical>
+                </position_sensing>
+                <velocity_sensing>
+                    <horizontal>
+                        <noise type="gaussian">
+                            <mean>0.0</mean>
+                            <stddev>0.01</stddev>
+                            <bias_mean>0.0</bias_mean>
+                            <bias_stddev>0.0</bias_stddev>
+                        </noise>
+                    </horizontal>
+                    <vertical>
+                        <noise type="gaussian">
+                            <mean>0.0</mean>
+                            <stddev>0.01</stddev>
+                            <bias_mean>0.0</bias_mean>
+                            <bias_stddev>0.0</bias_stddev>
+                        </noise>
+                    </vertical>
+                </velocity_sensing>
+            </gps>
             <plugin name="gps_plugin" filename="libgazebo_ros_gps_sensor.so">
                 <ros>

Commit message: refactor wheels with steering Knuckle, hub

File: ros2_ws/src/robot_description/urdf/fendt/fendt.urdf.xacro (robot description, xacro)
@@ -171,14 +171,17 @@
                 o_rpy="0 0 0"/>
     </link>
-    <joint name="front_axle_roll_joint" type="fixed">
+    <joint name="front_axle_roll_joint" type="revolute">
         <parent link="chassis"/>
         <child link="front_axle"/>
         <origin xyz="${front_axle_origin_x} 0 ${front_axle_origin_z}" rpy="0 0 0"/>
+        <axis xyz="1 0 0"/>
+        <limit lower="-0.1745329252" upper="0.1745329252" effort="3000.0" velocity="0.5"/>
+        <dynamics damping="80.0" friction="8.0"/>
     </joint>
     <!-- ===== Wheels ===== -->
-    <xacro:wheel name="rear_left_wheel"  parent="rear_axle"  x="0.0" y="${ wheel_y_distance}" z="0.0" radius="${wheel_rad_rear}" width="${wheel_width_r}" mass="${wheel_weight_r}"/>
-    <xacro:wheel name="rear_right_wheel" parent="rear_axle"  x="0.0" y="${-wheel_y_distance}" z="0.0" radius="${wheel_rad_rear}" width="${wheel_width_r}" mass="${wheel_weight_r}"/>
-    <xacro:steerable_wheel name="front_left_wheel"  parent="front_axle" x="0.0" y="${ wheel_y_distance}" z="0.0" radius="${wheel_rad_front}" width="${wheel_width_f}" mass="${wheel_weight_f}" steer_limit="${front_steer_limit}"/>
-    <xacro:steerable_wheel name="front_right_wheel" parent="front_axle" x="0.0" y="${-wheel_y_distance}" z="0.0" radius="${wheel_rad_front}" width="${wheel_width_f}" mass="${wheel_weight_f}" steer_limit="${front_steer_limit}"/>
+    <xacro:wheel name="rear_left_wheel"  parent="rear_axle"  x="0.0" y="${wheel_y_distance - (wheel_width_r/2.0)}" z="0.0" radius="${wheel_rad_rear}" width="${wheel_width_r}" mass="${wheel_weight_r}" axle_radius="${axle_rad_rear}" pivot_y_offset="${wheel_width_r/2.0}"/>
+    <xacro:wheel name="rear_right_wheel" parent="rear_axle"  x="0.0" y="${-wheel_y_distance + (wheel_width_r/2.0)}" z="0.0" radius="${wheel_rad_rear}" width="${wheel_width_r}" mass="${wheel_weight_r}" axle_radius="${axle_rad_rear}" pivot_y_offset="${-wheel_width_r/2.0}"/>
+    <xacro:steerable_wheel name="front_left_wheel"  parent="front_axle" x="0.0" y="${wheel_y_distance - (wheel_width_f/2.0)}" z="0.0" radius="${wheel_rad_front}" width="${wheel_width_f}" mass="${wheel_weight_f}" steer_limit="${front_steer_limit}" axle_radius="${axle_rad_front}" pivot_y_offset="${wheel_width_f/2.0}"/>
+    <xacro:steerable_wheel name="front_right_wheel" parent="front_axle" x="0.0" y="${-wheel_y_distance + (wheel_width_f/2.0)}" z="0.0" radius="${wheel_rad_front}" width="${wheel_width_f}" mass="${wheel_weight_f}" steer_limit="${front_steer_limit}" axle_radius="${axle_rad_front}" pivot_y_offset="${-wheel_width_f/2.0}"/>
     <!-- ===== Sensors ===== -->
     <link name="laser_frame"/>

File: ros2_ws/src/robot_description/urdf/fendt/fendt_gazebo.urdf.xacro (robot description, xacro)
@@ -20,4 +20,28 @@
     <gazebo reference="front_axle">
         <material>Gazebo/DarkGrey</material>
+    </gazebo>
+    <gazebo reference="rear_left_wheel_knuckle">
+        <material>Gazebo/DarkGrey</material>
+    </gazebo>
+    <gazebo reference="rear_right_wheel_knuckle">
+        <material>Gazebo/DarkGrey</material>
+    </gazebo>
+    <gazebo reference="front_left_wheel_knuckle">
+        <material>Gazebo/DarkGrey</material>
+    </gazebo>
+    <gazebo reference="front_right_wheel_knuckle">
+        <material>Gazebo/DarkGrey</material>
+    </gazebo>
+    <gazebo reference="rear_left_wheel_hub">
+        <material>Gazebo/Red</material>
+    </gazebo>
+    <gazebo reference="rear_right_wheel_hub">
+        <material>Gazebo/Red</material>
+    </gazebo>
+    <gazebo reference="front_left_wheel_hub">
+        <material>Gazebo/Red</material>
+    </gazebo>
+    <gazebo reference="front_right_wheel_hub">
+        <material>Gazebo/Red</material>
     </gazebo>
     <gazebo reference="rear_left_wheel">

File: ros2_ws/src/robot_description/urdf/fendt/wheels.xacro (robot description, xacro)
@@ -1,53 +1,60 @@
 <?xml version="1.0"?>
 <robot xmlns:xacro="http://www.ros.org/wiki/xacro">
-  <!-- ===== Wheel Macro ===== -->
-  <xacro:macro name="wheel" params="name parent x y z radius width mass:=50.0">
-    <link name="${name}">
+  <!-- ===== Rear Wheel Macro (axle -> knuckle -> hub -> tire) ===== -->
+  <xacro:macro name="wheel" params="name parent x y z radius width mass:=50.0 axle_radius:=0.13 pivot_y_offset:=0.0">
+    <xacro:property name="knuckle_length" value="${width + 0.04}"/>
+    <xacro:property name="hub_radius" value="${0.6 * radius}"/>
+    <xacro:property name="hub_length" value="${width + 0.02}"/>
+    <link name="${name}_knuckle">
+      <visual>
+        <origin xyz="0 ${pivot_y_offset} 0" rpy="1.57079632679 0 0"/>
+        <geometry>
+          <cylinder radius="${axle_radius}" length="${knuckle_length}"/>
+        </geometry>
+        <material name="grey"/>
+      </visual>
+      <collision>
+        <origin xyz="0 ${pivot_y_offset} 0" rpy="1.57079632679 0 0"/>
+        <geometry>
+          <cylinder radius="${axle_radius}" length="${knuckle_length}"/>
+        </geometry>
+      </collision>
+      <xacro:cylinder_inertia m="${0.1 * mass}"
+                              r="${axle_radius}"
+                              l="${knuckle_length}"
+                              o_xyz="0 ${pivot_y_offset} 0"
+                              o_rpy="0 0 0"/>
+    </link>
+    <joint name="${name}_knuckle_joint" type="fixed">
+      <parent link="${parent}"/>
+      <child link="${name}_knuckle"/>
+      <origin xyz="${x} ${y} ${z}" rpy="0 0 0"/>
+    </joint>
+    <link name="${name}_hub">
       <visual>
         <origin xyz="0 0 0" rpy="1.57079632679 0 0"/>
         <geometry>
-          <cylinder radius="${radius}" length="${width}"/>
+          <cylinder radius="${hub_radius}" length="${hub_length}"/>
         </geometry>
-        <material name="black"/>
+        <material name="red"/>
       </visual>
       <collision>
         <origin xyz="0 0 0" rpy="1.57079632679 0 0"/>
         <geometry>
-          <cylinder radius="${radius}" length="${width}"/>
+          <cylinder radius="${hub_radius}" length="${hub_length}"/>
         </geometry>
       </collision>
-      <xacro:cylinder_inertia m="${mass}"
-                              r="${radius}"
-                              l="${width}"
+      <xacro:cylinder_inertia m="${0.2 * mass}"
+                              r="${hub_radius}"
+                              l="${hub_length}"
                               o_xyz="0 0 0"
                               o_rpy="0 0 0"/>
     </link>
     <joint name="${name}_joint" type="continuous">
-      <parent link="${parent}"/>
-      <child link="${name}"/>
-      <origin xyz="${x} ${y} ${z}" rpy="0 0 0"/>
+      <parent link="${name}_knuckle"/>
+      <child link="${name}_hub"/>
+      <origin xyz="0 ${pivot_y_offset} 0" rpy="0 0 0"/>
       <axis xyz="0 1 0"/>
       <dynamics damping="12.0" friction="2.0"/>
-    </joint>
-  </xacro:macro>
-  <xacro:macro name="steerable_wheel" params="name parent x y z radius width mass:=50.0 steer_limit:=0.9599310886 mimic_joint:='' mimic_multiplier:=1.0">
-    <link name="${name}_steer">
-      <!-- Keep a physical steering knuckle link so Gazebo doesn't prune the front wheel chain -->
-      <inertial>
-        <mass value="1.0"/>
-        <origin xyz="0 0 0" rpy="0 0 0"/>
-        <inertia ixx="0.001" ixy="0.0" ixz="0.0" iyy="0.001" iyz="0.0" izz="0.001"/>
-      </inertial>
-    </link>
-    <joint name="${name}_steer_joint" type="revolute">
-      <parent link="${parent}"/>
-      <child link="${name}_steer"/>
-      <origin xyz="${x} ${y} ${z}" rpy="0 0 0"/>
-      <axis xyz="0 0 1"/>
-      <limit lower="${-steer_limit}" upper="${steer_limit}" effort="2000.0" velocity="1.5"/>
-      <xacro:if value="${mimic_joint != ''}">
-        <mimic joint="${mimic_joint}" multiplier="${mimic_multiplier}" offset="0.0"/>
-      </xacro:if>
-      <dynamics damping="150.0" friction="15.0"/>
     </joint>
     <link name="${name}">
@@ -65,5 +72,5 @@
         </geometry>
       </collision>
-      <xacro:cylinder_inertia m="${mass}"
+      <xacro:cylinder_inertia m="${0.7 * mass}"
                               r="${radius}"
                               l="${width}"
@@ -71,11 +78,97 @@
                               o_rpy="0 0 0"/>
     </link>
-    <joint name="${name}_joint" type="continuous">
-      <parent link="${name}_steer"/>
+    <joint name="${name}_tire_joint" type="fixed">
+      <parent link="${name}_hub"/>
       <child link="${name}"/>
       <origin xyz="0 0 0" rpy="0 0 0"/>
+    </joint>
+  </xacro:macro>
+  <xacro:macro name="steerable_wheel" params="name parent x y z radius width mass:=50.0 steer_limit:=0.9599310886 mimic_joint:='' mimic_multiplier:=1.0 axle_radius:=0.13 pivot_y_offset:=0.0">
+    <xacro:property name="knuckle_length" value="${width + 0.04}"/>
+    <xacro:property name="hub_radius" value="${0.6 * radius}"/>
+    <xacro:property name="hub_length" value="${width + 0.02}"/>
+    <link name="${name}_knuckle">
+      <visual>
+        <origin xyz="0 ${pivot_y_offset} 0" rpy="1.57079632679 0 0"/>
+        <geometry>
+          <cylinder radius="${axle_radius}" length="${knuckle_length}"/>
+        </geometry>
+        <material name="grey"/>
+      </visual>
+      <collision>
+        <origin xyz="0 ${pivot_y_offset} 0" rpy="1.57079632679 0 0"/>
+        <geometry>
+          <cylinder radius="${axle_radius}" length="${knuckle_length}"/>
+        </geometry>
+      </collision>
+      <xacro:cylinder_inertia m="${0.1 * mass}"
+                              r="${axle_radius}"
+                              l="${knuckle_length}"
+                              o_xyz="0 ${pivot_y_offset} 0"
+                              o_rpy="0 0 0"/>
+    </link>
+    <joint name="${name}_steer_joint" type="revolute">
+      <parent link="${parent}"/>
+      <child link="${name}_knuckle"/>
+      <origin xyz="${x} ${y} ${z}" rpy="0 0 0"/>
+      <axis xyz="0 0 1"/>
+      <limit lower="${-steer_limit}" upper="${steer_limit}" effort="2000.0" velocity="1.5"/>
+      <xacro:if value="${mimic_joint != ''}">
+        <mimic joint="${mimic_joint}" multiplier="${mimic_multiplier}" offset="0.0"/>
+      </xacro:if>
+      <dynamics damping="150.0" friction="15.0"/>
+    </joint>
+    <link name="${name}_hub">
+      <visual>
+        <origin xyz="0 0 0" rpy="1.57079632679 0 0"/>
+        <geometry>
+          <cylinder radius="${hub_radius}" length="${hub_length}"/>
+        </geometry>
+        <material name="red"/>
+      </visual>
+      <collision>
+        <origin xyz="0 0 0" rpy="1.57079632679 0 0"/>
+        <geometry>
+          <cylinder radius="${hub_radius}" length="${hub_length}"/>
+        </geometry>
+      </collision>
+      <xacro:cylinder_inertia m="${0.2 * mass}"
+                              r="${hub_radius}"
+                              l="${hub_length}"
+                              o_xyz="0 0 0"
+                              o_rpy="0 0 0"/>
+    </link>
+    <joint name="${name}_joint" type="continuous">
+      <parent link="${name}_knuckle"/>
+      <child link="${name}_hub"/>
+      <origin xyz="0 ${pivot_y_offset} 0" rpy="0 0 0"/>
       <axis xyz="0 1 0"/>
       <dynamics damping="10.0" friction="1.5"/>
     </joint>
+    <link name="${name}">
+      <visual>
+        <origin xyz="0 0 0" rpy="1.57079632679 0 0"/>
+        <geometry>
+          <cylinder radius="${radius}" length="${width}"/>
+        </geometry>
+        <material name="black"/>
+      </visual>
+      <collision>
+        <origin xyz="0 0 0" rpy="1.57079632679 0 0"/>
+        <geometry>
+          <cylinder radius="${radius}" length="${width}"/>
+        </geometry>
+      </collision>
+      <xacro:cylinder_inertia m="${0.7 * mass}"
+                              r="${radius}"
+                              l="${width}"
+                              o_xyz="0 0 0"
+                              o_rpy="0 0 0"/>
+    </link>
+    <joint name="${name}_tire_joint" type="fixed">
+      <parent link="${name}_hub"/>
+      <child link="${name}"/>
+      <origin xyz="0 0 0" rpy="0 0 0"/>
+    </joint>
   </xacro:macro>
 </robot>

Commit message: refactor wheels with steering Knuckle, hub 2

File: ros2_ws/src/robot_description/urdf/fendt/fendt.urdf.xacro (robot description, xacro)
@@ -18,5 +18,5 @@
     <xacro:property name="wheel_rad_front" value="0.59"/>
     <xacro:property name="wheel_width_f" value="0.44"/>
-    <xacro:property name="front_steer_limit" value="0.7853981634"/>
+    <xacro:property name="front_steer_limit" value="0.6108652382"/>
     <xacro:property name="axle_rad_front" value="0.13"/>
     <xacro:property name="axle_len_front" value="${wheel_track-wheel_width_f}"/>
@@ -34,5 +34,5 @@
     <xacro:property name="axle_to_r_body" value="0.20"/>
     <xacro:property name="box_len_r_body" value="${axle_to_r_body + half_wheelbase}"/>
-    <xacro:property name="box_width_r_body" value="${full_width-(2*wheel_width_r)}"/>
+    <xacro:property name="box_width_r_body" value="${full_width-2*wheel_width_r-0.10}"/>
     <xacro:property name="box_height_r_body" value="${full_height-bottom_clearance}"/>
     <xacro:property name="weight_f_body" value="150"/>
@@ -171,5 +171,5 @@
                 o_rpy="0 0 0"/>
     </link>
-    <joint name="front_axle_roll_joint" type="revolute">
+    <joint name="front_axle_roll_joint" type="fixed">
         <parent link="chassis"/>
         <child link="front_axle"/>

File: ros2_ws/src/robot_description/urdf/fendt/fendt_gazebo.urdf.xacro (robot description, xacro)
@@ -13,5 +13,5 @@
     </gazebo>
     <gazebo reference="rear_body">
-        <material>Gazebo/Red</material>
+        <material>Gazebo/White</material>
     </gazebo>
     <gazebo reference="rear_axle">

Commit message: refactor wheels with steering Knuckle, hub 3

File: ros2_ws/src/robot_description/urdf/fendt/fendt.urdf.xacro (robot description, xacro)
@@ -187,5 +187,5 @@
     <link name="laser_frame"/>
     <joint name="laser_joint" type="fixed">
-        <parent link="rear_body"/>
+        <parent link="base_link"/>
         <child link="laser_frame"/>
         <origin xyz="0.0 0.0 ${laser_origin_z}" rpy="0 0 0"/>
