Commit message: fix drift issue

File: ros2_ws/src/robot_description/urdf/fendt/fendt.urdf.xacro (robot description, xacro)
@@ -165,5 +165,5 @@
         </collision>
         <xacro:cylinder_inertia
-                m="${wheel_weight_f}"
+                m="${weight_f_axle}"
                 r="${axle_rad_front}"
                 l="${axle_len_front}"

File: ros2_ws/src/robot_description/urdf/fendt/fendt_gazebo.urdf.xacro (robot description, xacro)
@@ -8,4 +8,8 @@
         <mu1>0.5</mu1>
         <mu2>0.5</mu2>
+        <velocity_decay>
+            <linear>0.2</linear>
+            <angular>0.2</angular>
+        </velocity_decay>
     </gazebo>
     <gazebo reference="front_body">
@@ -47,29 +51,37 @@
     <gazebo reference="rear_left_wheel">
         <material>Gazebo/Black</material>
-        <mu1>2.5</mu1>
-        <mu2>2.5</mu2>
-        <kp>1e7</kp>
-        <kd>500.0</kd>
+        <mu1>3.2</mu1>
+        <mu2>3.2</mu2>
+        <kp>1e7</kp>
+        <kd>1000.0</kd>
+        <slip1>0.0</slip1>
+        <slip2>0.0</slip2>
     </gazebo>
     <gazebo reference="rear_right_wheel">
         <material>Gazebo/Black</material>
-        <mu1>2.5</mu1>
-        <mu2>2.5</mu2>
-        <kp>1e7</kp>
-        <kd>500.0</kd>
+        <mu1>3.2</mu1>
+        <mu2>3.2</mu2>
+        <kp>1e7</kp>
+        <kd>1000.0</kd>
+        <slip1>0.0</slip1>
+        <slip2>0.0</slip2>
     </gazebo>
     <gazebo reference="front_left_wheel">
         <material>Gazebo/Black</material>
-        <mu1>2.5</mu1>
-        <mu2>2.5</mu2>
-        <kp>1e7</kp>
-        <kd>500.0</kd>
+        <mu1>3.2</mu1>
+        <mu2>3.2</mu2>
+        <kp>1e7</kp>
+        <kd>1000.0</kd>
+        <slip1>0.0</slip1>
+        <slip2>0.0</slip2>
     </gazebo>
     <gazebo reference="front_right_wheel">
         <material>Gazebo/Black</material>
-        <mu1>2.5</mu1>
-        <mu2>2.5</mu2>
-        <kp>1e7</kp>
-        <kd>500.0</kd>
+        <mu1>3.2</mu1>
+        <mu2>3.2</mu2>
+        <kp>1e7</kp>
+        <kd>1000.0</kd>
+        <slip1>0.0</slip1>
+        <slip2>0.0</slip2>
     </gazebo>
     <gazebo reference="laser_frame">
@@ -129,5 +141,5 @@
                         <noise type="gaussian">
                             <mean>0.0</mean>
-                            <stddev>0.02</stddev>
+                            <stddev>0.0</stddev>
                             <bias_mean>0.0</bias_mean>
                             <bias_stddev>0.0</bias_stddev>
@@ -137,5 +149,5 @@
                         <noise type="gaussian">
                             <mean>0.0</mean>
-                            <stddev>0.03</stddev>
+                            <stddev>0.0</stddev>
                             <bias_mean>0.0</bias_mean>
                             <bias_stddev>0.0</bias_stddev>
@@ -147,5 +159,5 @@
                         <noise type="gaussian">
                             <mean>0.0</mean>
-                            <stddev>0.01</stddev>
+                            <stddev>0.0</stddev>
                             <bias_mean>0.0</bias_mean>
                             <bias_stddev>0.0</bias_stddev>
@@ -155,5 +167,5 @@
                         <noise type="gaussian">
                             <mean>0.0</mean>
-                            <stddev>0.01</stddev>
+                            <stddev>0.0</stddev>
                             <bias_mean>0.0</bias_mean>
                             <bias_stddev>0.0</bias_stddev>

File: ros2_ws/src/robot_description/urdf/fendt/wheels.xacro (robot description, xacro)
@@ -56,5 +56,5 @@
       <origin xyz="0 ${pivot_y_offset} 0" rpy="0 0 0"/>
       <axis xyz="0 1 0"/>
-      <dynamics damping="12.0" friction="2.0"/>
+      <dynamics damping="25.0" friction="6.0"/>
     </joint>
     <link name="${name}">
@@ -117,5 +117,5 @@
         <mimic joint="${mimic_joint}" multiplier="${mimic_multiplier}" offset="0.0"/>
       </xacro:if>
-      <dynamics damping="150.0" friction="15.0"/>
+      <dynamics damping="300.0" friction="45.0"/>
     </joint>
     <link name="${name}_hub">
@@ -144,5 +144,5 @@
       <origin xyz="0 ${pivot_y_offset} 0" rpy="0 0 0"/>
       <axis xyz="0 1 0"/>
-      <dynamics damping="10.0" friction="1.5"/>
+      <dynamics damping="20.0" friction="5.0"/>
     </joint>
     <link name="${name}">

Commit message: update md

File: ros2_ws/src/robot_description/urdf/fendt/fendt.urdf.xacro (robot description, xacro)
@@ -31,5 +31,5 @@
     <xacro:property name="box_len_f_body" value="${axle_to_front_f_body + half_wheelbase}"/>
     <xacro:property name="box_width_f_body" value="0.60"/>
-    <xacro:property name="box_height_f_body" value="0.50"/>
+    <xacro:property name="box_height_f_body" value="0.60"/>
     <xacro:property name="axle_to_r_body" value="0.20"/>
     <xacro:property name="box_len_r_body" value="${axle_to_r_body + half_wheelbase}"/>

Commit message: update rear body height

File: ros2_ws/src/robot_description/urdf/fendt/fendt.urdf.xacro (robot description, xacro)
@@ -35,5 +35,5 @@
     <xacro:property name="box_len_r_body" value="${axle_to_r_body + half_wheelbase}"/>
     <xacro:property name="box_width_r_body" value="${full_width-2*wheel_width_r-0.10}"/>
-    <xacro:property name="box_height_r_body" value="${full_height-bottom_clearance}"/>
+    <xacro:property name="box_height_r_body" value="${full_height-bottom_clearance - chassis_origin_z}"/>
     <xacro:property name="weight_f_body" value="150"/>
     <xacro:property name="weight_r_body" value="250"/>
@@ -51,5 +51,5 @@
     <xacro:property name="front_axle_origin_z" value="${wheel_rad_front - (bottom_clearance+chassis_origin_z)}"/>
     <xacro:property name="rear_body_origin_x" value="${-box_len_r_body/2.0}"/>
-    <xacro:property name="rear_body_origin_z" value="${box_height_r_body/2.0 - chassis_origin_z}"/>
+    <xacro:property name="rear_body_origin_z" value="${box_height_r_body/2.0}"/>
     <xacro:property name="front_body_origin_x" value="${box_len_f_body/2.0}"/>
     <xacro:property name="front_body_origin_z" value="${box_height_f_body/2.0 + chassis_origin_z}"/>
